File: Board/Power.kicad_sch (KiCad schematic)
At the start: 81 parts, among them J2 DCJ0202, Q4 IRLML5203

Commit message: Ultipet 1.0A final
Parts:
- removed C63: 22u, cbm_ultipet_v1:C0805, symbol cbm_ultipet_v1-eagle-import:C-EUC0805
- removed R23: 10k, cbm_ultipet_v1:0207_2V, symbol cbm_ultipet_v1-eagle-import:R-EU_0207/2V
- removed U$17: AP2132BB, cbm_ultipet_v1:PSOP-8-FIXED, symbol cbm_ultipet_v1-eagle-import:AP2132BB
- added C127, C128, C63, C85: 100n, cbm_ultipet_v1:C0603, symbol cbm_ultipet_v1-eagle-import:C-EUC0603
Connections:
- net V25 is gone; now on net 3.3V: C101.1, C104.1, C109.1, C112.1, C121.1, C123.1, C64.1, U$16.2 (EN)
- net 3.3V: now also C127.1, C128.1, C63.1, C85.1
- net GND: now also C127.2, C128.2, C63.2, C85.2
- net VCC: now also SW1.5
- net VCCIN: now also SW1.4

Commit message: ultipet 1.1a board
Parts:
- SW1: footprint Footprints:SW_E-Switch-400AWMDPxR1M1x -> Footprints:SW_E-Switch-400-combined
Connections:
- net 3.3V renamed V33
Other:
- note added: "1.1A: - change footprint of power switch to a combined one"
- note added: "CBM-ULTIPET-V1.1A"
- note added: "CSA-ULTIPET-V1.1A-20240603"
- note removed: "CBM-ULTIPET-V1.0A"
- note removed: "CSA-ULTIPET-V1.0A-20240104"
Changed lines of the file:
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@@
 		)
 	)
-	(text "CBM-ULTIPET-V1.0A"
+	(text "CBM-ULTIPET-V1.1A"
 		(exclude_from_sim no)
 		(at 208.28 195.58 0)
@@
 		)
 	)
+	(text "1.1A:\n- change footprint of power switch to a combined one"
+		(exclude_from_sim no)
+		(at 210.312 184.658 0)
+		(effects
+			(font
+				(size 2 2)
+			)
+			(justify left)
+		)
+	)
 	(text "(C) A. Fachat"
 		(exclude_from_sim no)
@@
 		)
 	)
-	(text "CSA-ULTIPET-V1.0A-20240104"
+	(text "CSA-ULTIPET-V1.1A-20240603"
 		(exclude_from_sim no)
 		(at 208.28 218.44 0)
@@
 			)
 		)
-		(property "Value" "3.3V"
+		(property "Value" "V33"
 			(at 232.664 136.144 0)
 			(effects
@@
 			)
 		)
-		(property "Value" "3.3V"
+		(property "Value" "V33"
 			(at 47.244 143.764 0)
 			(effects
@@
 			)
 		)
-		(property "Value" "VDD"
+		(property "Value" "V33"
 			(at 25.4 170.18 90)
 			(effects
@@
 			)
 		)
-		(property "Footprint" "Footprints:SW_E-Switch-400AWMDPxR1M1x"
+		(property "Footprint" "Footprints:SW_E-Switch-400-combined"
 			(at 93.98 41.91 0)
 			(effects

Commit message: diverse fixes
Parts:
- added C152, C155: 100n, cbm_ultipet_v1:C0603, symbol cbm_ultipet_v1-eagle-import:C-EUC0603
- added C153: 47u, cbm_ultipet_v1:E2,5-6, symbol cbm_ultipet_v1-eagle-import:CPOL-EUE2.5-6
- added C154: 22u, cbm_ultipet_v1:C0805, symbol cbm_ultipet_v1-eagle-import:C-EUC0805
- added JP19: ~, cbm_ultipet_v1:JP4, symbol cbm_ultipet_v1-eagle-import:JP4E
- added JP8: JP1E, cbm_ultipet_v1:JP1, symbol cbm_ultipet_v1-eagle-import:JP1E
- added R17, R26: 390, cbm_ultipet_v1:0207_2V, symbol cbm_ultipet_v1-eagle-import:R-EU_0207/2V
- added U$17: LDI1117, cbm_ultipet_v1:SOT223, symbol cbm_ultipet_v1-eagle-import:LDI1117
Connections:
- net GND: now also C152.2, C153.-, C154.2, C155.2, JP19.3, JP8.2, U$17.1 (GND)
- net V33: now also R26.2
- net VCC: now also C152.1, C153.+, JP8.1, U$17.3 (VI)
- new net: JP19.1, R26.1
- new net: JP19.4, R17.1
- new net KEYLOCK_LED: JP19.2
- new net V33IO: C154.1, C155.1, U$17.2 (VO)
Other:
- note added: "1.1A: - change footprint of power switch to a combined one 1.2A: - add LED connector - add 3.3V for I/O"
- note added: "3.3V Generation for I/O"
- note added: "CBM-ULTIPET-V1.2A"
- note added: "CSA-ULTIPET-V1.2A-20241010"
- note added: "LED Connector for Power and Shift-Lock state"
- note removed: "1.1A: - change footprint of power switch to a combined one"
- note removed: "CBM-ULTIPET-V1.1A"
- note removed: "CSA-ULTIPET-V1.1A-20240603"
- moved on the sheet: C5, C6, C64, C65, C66, C7, C70, C8, R24, S1

Commit message: various fixes as documented in github issues
Parts:
- R26: value 390 -> 100
Other:
- note added: "Resistor values for 2V fwd voltage, 20mA current LEDs"
Changed lines of the file:
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@@
 		)
 	)
+	(text "Resistor values for\n2V fwd voltage, \n20mA current LEDs\n"
+		(exclude_from_sim no)
+		(at 189.992 22.606 0)
+		(effects
+			(font
+				(size 1.27 1.27)
+			)
+		)
+	)
 	(text "DS1818"
 		(exclude_from_sim no)
@@
 			)
 		)
-		(property "Value" "390"
+		(property "Value" "100"
 			(at 186.182 40.64 0)
 			(effects

Commit message: more fixes
Connections:
- net VCC: no longer SW1.5
- net VCCIN: now also SW1.3, SW1.5; no longer SW1.1, SW1.4
Changed lines of the file:
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@@
 	)
 	(junction
-		(at 104.14 48.26)
-		(diameter 0)
-		(color 0 0 0 0)
-	)
-	(junction
 		(at 152.4 119.38)
 		(diameter 0)
@@
 	)
 	(junction
-		(at 85.09 45.72)
-		(diameter 0)
-		(color 0 0 0 0)
-	)
-	(junction
 		(at 88.9 104.14)
 		(diameter 0)
@@
 	)
 	(junction
+		(at 85.09 50.8)
+		(diameter 0)
+		(color 0 0 0 0)
+	)
+	(junction
 		(at 151.13 175.26)
 		(diameter 0)
@@
 	(wire
 		(pts
+			(xy 85.09 66.04) (xy 85.09 50.8)
+		)
+		(stroke
+			(width 0)
+			(type default)
+		)
+	)
+	(wire
+		(pts
 			(xy 231.14 110.49) (xy 231.14 107.95)
 		)
@@
 	(wire
 		(pts
-			(xy 85.09 57.15) (xy 85.09 45.72)
+			(xy 85.09 45.72) (xy 85.09 50.8)
 		)
 		(stroke
@@
 	(wire
 		(pts
-			(xy 90.17 57.15) (xy 85.09 57.15)
-		)
-		(stroke
-			(width 0)
-			(type default)
-		)
-	)
-	(wire
-		(pts
 			(xy 101.6 93.98) (xy 111.76 93.98)
 		)
@@
 	(wire
 		(pts
-			(xy 99.06 88.9) (xy 109.22 88.9)
+			(xy 107.95 66.04) (xy 85.09 66.04)
 		)
 		(stroke
-			(width 0.1524)
-			(type solid)
+			(width 0)
+			(type default)
 		)
 	)
 	(wire
 		(pts
-			(xy 104.14 59.69) (xy 104.14 48.26)
+			(xy 99.06 88.9) (xy 109.22 88.9)
 		)
 		(stroke
-			(width 0)
-			(type default)
+			(width 0.1524)
+			(type solid)
 		)
 	)
@@
 	(wire
 		(pts
+			(xy 102.87 59.69) (xy 107.95 59.69)
+		)
+		(stroke
+			(width 0)
+			(type default)
+		)
+	)
+	(wire
+		(pts
 			(xy 238.76 110.49) (xy 231.14 110.49)
 		)
@@
 	(wire
 		(pts
+			(xy 107.95 59.69) (xy 107.95 66.04)
+		)
+		(stroke
+			(width 0)
+			(type default)
+		)
+	)
+	(wire
+		(pts
 			(xy 238.76 152.4) (xy 238.76 154.94)
 		)
@@
 	(wire
 		(pts
-			(xy 102.87 59.69) (xy 104.14 59.69)
-		)
-		(stroke
-			(width 0)
-			(type default)
-		)
-	)
-	(wire
-		(pts
 			(xy 81.28 104.14) (xy 78.74 104.14)
 		)
@@
 	(wire
 		(pts
+			(xy 85.09 50.8) (xy 90.17 50.8)
+		)
+		(stroke
+			(width 0)
+			(type default)
+		)
+	)
+	(wire
+		(pts
 			(xy 106.68 160.02) (xy 114.3 160.02)
 		)
@@
 	(wire
 		(pts
-			(xy 104.14 48.26) (xy 105.41 48.26)
-		)
-		(stroke
-			(width 0)
-			(type default)
-		)
-	)
-	(wire
-		(pts
 			(xy 88.9 109.22) (xy 88.9 104.14)
 		)
@@
 	(wire
 		(pts
-			(xy 102.87 48.26) (xy 104.14 48.26)
+			(xy 102.87 48.26) (xy 105.41 48.26)
 		)
 		(stroke
@@
 		)
 	)
-	(wire
-		(pts
-			(xy 85.09 45.72) (xy 90.17 45.72)
-		)
-		(stroke
-			(width 0)
-			(type default)
-		)
-	)

Commit message: more layout work
Parts:
- removed C22, C24: 0.1u, cbm_ultipet_v1:C0603, symbol cbm_ultipet_v1-eagle-import:C-EUC0603
Changed lines of the file:
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@@
 	)
 	(symbol
-		(lib_id "cbm_ultipet_v1-eagle-import:C-EUC0603")
-		(at 60.96 99.06 0)
-		(unit 1)
-		(exclude_from_sim no)
-		(in_bom yes)
-		(on_board yes)
-		(dnp no)
-		(property "Reference" "C22"
-			(at 62.484 98.679 0)
-			(effects
-				(font
-					(size 1.778 1.5113)
-				)
-				(justify left bottom)
-			)
-		)
-		(property "Value" "0.1u"
-			(at 62.484 103.759 0)
-			(effects
-				(font
-					(size 1.778 1.5113)
-				)
-				(justify left bottom)
-			)
-		)
-		(property "Footprint" "cbm_ultipet_v1:C0603"
-			(at 60.96 99.06 0)
-			(effects
-				(font
-					(size 1.27 1.27)
-				)
-				(hide yes)
-			)
-		)
-		(property "Datasheet" ""
-			(at 60.96 99.06 0)
-			(effects
-				(font
-					(size 1.27 1.27)
-				)
-				(hide yes)
-			)
-		)
-		(property "Description" ""
-			(at 60.96 99.06 0)
-			(effects
-				(font
-					(size 1.27 1.27)
-				)
-				(hide yes)
-			)
-		)
-		(pin "2"
-		)
-		(pin "1"
-		)
-		(instances
-			(project "cbm_ultipet_v1"
-				(path "/4dd2dd78-173f-4b46-8cce-4ed940435c94/f2a7836e-baa5-4eed-9e59-e26d91b4d1a6"
-					(reference "C22")
-					(unit 1)
-				)
-			)
-		)
-	)
-	(symbol
 		(lib_id "cbm_ultipet_v1-eagle-import:GND")
 		(at 106.68 35.56 0)
@@
 					(unit 1)
 				)
-			)
-		)
-	)
-	(symbol
-		(lib_id "cbm_ultipet_v1-eagle-import:C-EUC0603")
-		(at 81.28 99.06 0)
-		(unit 1)
-		(exclude_from_sim no)
-		(in_bom yes)
-		(on_board yes)
-		(dnp no)
-		(property "Reference" "C24"
-			(at 82.804 98.679 0)
-			(effects
-				(font
-					(size 1.778 1.5113)
-				)
-				(justify left bottom)
-			)
-		)
-		(property "Value" "0.1u"
-			(at 82.804 103.759 0)
-			(effects
-				(font
-					(size 1.778 1.5113)
-				)
-				(justify left bottom)
-			)
-		)
-		(property "Footprint" "cbm_ultipet_v1:C0603"
-			(at 81.28 99.06 0)
-			(effects
-				(font
-					(size 1.27 1.27)
-				)
-				(hide yes)
-			)
-		)
-		(property "Datasheet" ""
-			(at 81.28 99.06 0)
-			(effects
-				(font
-					(size 1.27 1.27)
-				)
-				(hide yes)
-			)
-		)
-		(property "Description" ""
-			(at 81.28 99.06 0)
-			(effects
-				(font
-					(size 1.27 1.27)
-				)
-				(hide yes)
-			)
-		)
-		(pin "2"
-		)
-		(pin "1"
-		)
-		(instances
-			(project "cbm_ultipet_v1"
-				(path "/4dd2dd78-173f-4b46-8cce-4ed940435c94/f2a7836e-baa5-4eed-9e59-e26d91b4d1a6"
-					(reference "C24")
-					(unit 1)
-				)

Commit message: fixed power switch footprint that got replaced on some update
Parts:
- SW1: footprint Footprints:SW_E-Switch-400-combined -> Footprints:SW_E-Switch-400-combined2
Changed lines of the file:
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@@
 	(label "VCCIN"
 		(at 81.28 45.72 0)
-		(fields_autoplaced yes)
 		(effects
 			(font
@@
 	(label "VCCIN"
 		(at 33.02 40.64 90)
-		(fields_autoplaced yes)
 		(effects
 			(font
@@
 	(label "VCCIN"
 		(at 142.24 54.61 180)
-		(fields_autoplaced yes)
 		(effects
 			(font
@@
 			)
 		)
-		(property "Footprint" "Footprints:SW_E-Switch-400-combined"
+		(property "Footprint" "Footprints:SW_E-Switch-400-combined2"
 			(at 93.98 41.91 0)
 			(effects

Commit message: first work on r1.3
Connections:
- net VCC: now also R17.2
Changed lines of the file:
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@@
+	(wire
+		(pts
+			(xy 205.74 30.48) (xy 205.74 31.75)
+		)
+		(stroke
+			(width 0)
+			(type default)
+		)
+	)
 	(wire
 		(pts
