File: Board/Power.kicad_sch (KiCad schematic)
At the start: 90 parts, among them J15 2171800001

Commit message: rename U refs to UX*
Parts:
- renumbered U$16 to UX16, U$17 to UX17, U$26 to UX26, U$3 to UX3
Changed lines of the file:
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@@
 		(on_board yes)
 		(dnp no)
-		(property "Reference" "U$16"
+		(property "Reference" "UX16"
 			(at 269.24 27.94 0)
 			(effects
@@
 			(project "cbm_ultipet_v1"
 				(path "/4dd2dd78-173f-4b46-8cce-4ed940435c94/f2a7836e-baa5-4eed-9e59-e26d91b4d1a6"
-					(reference "U$16")
+					(reference "UX16")
 					(unit 1)
 				)
@@
 		(on_board yes)
 		(dnp no)
-		(property "Reference" "U$26"
+		(property "Reference" "UX26"
 			(at 138.43 44.45 90)
 			(effects
@@
 			(project "cbm_ultipet_v1"
 				(path "/4dd2dd78-173f-4b46-8cce-4ed940435c94/f2a7836e-baa5-4eed-9e59-e26d91b4d1a6"
-					(reference "U$26")
+					(reference "UX26")
 					(unit 1)
 				)
@@
 		(on_board yes)
 		(dnp no)
-		(property "Reference" "U$17"
+		(property "Reference" "UX17"
 			(at 251.46 133.985 0)
 			(effects
@@
 			(project "cbm_ultipet_v1"
 				(path "/4dd2dd78-173f-4b46-8cce-4ed940435c94/f2a7836e-baa5-4eed-9e59-e26d91b4d1a6"
-					(reference "U$17")
+					(reference "UX17")
 					(unit 1)
 				)
@@
 		(on_board yes)
 		(dnp no)
-		(property "Reference" "U$3"
+		(property "Reference" "UX3"
 			(at 251.46 89.535 0)
 			(effects
@@
 			(project "cbm_ultipet_v1"
 				(path "/4dd2dd78-173f-4b46-8cce-4ed940435c94/f2a7836e-baa5-4eed-9e59-e26d91b4d1a6"
-					(reference "U$3")
+					(reference "UX3")
 					(unit 1)
 				)

Commit message: some layout fixes, more parts
Parts:
- removed J15: 2171800001, cbm_ultipet_v1:MOLEX_2171800001, symbol Symbols:2171800001
- added U11: USB-C Power, cbm_ultipet_v1:USB-C-217180, symbol Symbols:USB-C-217180
- C38: value 22u -> 47u
Connections:
- net GND: now also U11.A1B12 (GND1), U11.B1A12 (GND2), U11.S1 (SHLD1), U11.S2 (SHLD2), U11.S3 (SHLD3), U11.S4 (SHLD4)
- net UCD+: now also U11.A6 (AD+), U11.B6 (BD+)
- net UCD-: now also U11.A7 (AD-), U11.B7 (BD-)
- net VCCIN: now also U11.A4B9 (VBUS1), U11.B4A9 (VBUS2)
- net at R42.2: now also U11.A5 (ACC)
- net at R41.2: now also U11.B5 (BCC)
