File: Board/CPU,_FPGA,_FRAM.kicad_sch (KiCad schematic)
At the start: 21 parts, among them IC1 RAMSOCK32TO512KSOP, IC3 74125D, IC7 74138D

Commit message: Ultipet 1.0A final
Parts:
- removed U$2: XC3S100E, cbm_ultipet_v1:TQFP144, symbol cbm_ultipet_v1-eagle-import:XC3S100E
- added J1, J3, J4, J5: Conn_01x01_Pin, Connector_PinHeader_2.54mm:PinHeader_1x01_P2.54mm_Vertical, symbol Connector:Conn_01x01_Pin
- added U$19: XC6SLX9-TQG144, cbm_ultipet_v1:TQFP144, symbol micropet_v3-eagle-import:XC6SLX9-TQG144
- added U1: 74LVC1G04, Package_TO_SOT_SMD:SOT-23-5, symbol 74xGxx:74LVC1G04
Connections:
- net V25 is gone; now on net V33: R25.2, U$7.4 (VCC)
- net /BE_DOUT: now also U$19.133 (IO_L34N_GCLK18_0)
- net /BE_OUT: now also U$19.132 (IO_L35P_GCLK17_0)
- net /FRAMSEL: now also U$19.120 (IO_L62N_VREF_0)
- net /IOSEL: now also U$19.134 (IO_L34P_GCLK19_0)
- net /IRQ: now also J4.1 (Pin_1), U$19.23 (IO_L41N_GCLK26_3)
- net /LDAC: now also U$19.138 (IO_L4P_0)
- net /MEMSEL: now also U$19.112 (IO_L66P_SCP1_0)
- net /RAMCS/M1: now also U$19.59 (IO_L13N_D10_2); no longer IC3.6 (O)
- net /RAMWE: now also U$19.82 (IO_L45N_1)
- net /RES: now also U$19.117 (IO_L64P_SCP5_0)
- net 50M: now also U$19.123 (IO_L37N_GCLK12_0)
- net A0: now also U$19.17 (IO_L43P_GCLK23_3)
- net A1: now also U$19.56 (IO_L30P_GCLK1_D13_2)
- net A10: now also U$19.11 (IO_L49N_3)
- net A11: now also U$19.142 (IO_L2P_0)
- net A12: now also U$19.127 (IO_L36P_GCLK15_0)
- net A13: now also U$19.139 (IO_L3N_0)
- net A14: now also U$19.119 (IO_L63P_SCP7_0)
- net A15: now also U$19.131 (IO_L35N_GCLK16_0)
- net A2: now also U$19.45 (IO_L49N_D4_2)
- net A3: now also U$19.43 (IO_L62N_D6_2)
- net A4: now also U$19.44 (IO_L62P_D5_2)
- net A5: now also U$19.40 (IO_L64N_D9_2)
- net A6: now also U$19.41 (IO_L64P_D8_2)
- net A7: now also U$19.26 (IO_L37N_3)
- net A8: now also U$19.30 (IO_L36P_3)
- net A9: now also U$19.10 (IO_L50P_3)
- net BE_IN: now also U$19.118 (IO_L63N_SCP6_0)
- net BOUT: now also U$19.94 (IO_L40N_GCLK10_1)
- net C2PHI2: now also U$19.104 (IO_L1N_VREF_1)
- net C8PHI2: now also U$19.102 (IO_L32P_1)
- net CPHI2: now also U$19.114 (IO_L65N_SCP2_0)
- net D0: now also U$19.2 (IO_L83P_3)
- net D1: now also U$19.1 (IO_L83N_VREF_3)
- net D2: now also U$19.14 (IO_L44N_GCLK20_3)
- net D3: now also U$19.5 (IO_L52N_3)
- net D4: now also U$19.12 (IO_L49P_3)
- net D5: now also U$19.8 (IO_L51P_3)
- net D6: now also U$19.9 (IO_L50N_3)
- net D7: now also U$19.6 (IO_L52P_3)
- net DONE: now also U$19.71 (DONE_2); no longer U$1.40 (BE)
- net E: now also U$19.21 (IO_L42N_GCLK24_3)
- net EXTIO: now also U$19.115 (IO_L65P_SCP3_0)
- net FA15: now also U$19.140 (IO_L3P_0)
- net FA16: now also U$19.141 (IO_L2N_0)
- net FA17: now also U$19.143 (IO_L1N_VREF_0)
- net FA18: now also U$19.144 (IO_L1P_HSWAPEN_0)
- net FA19: now also U$19.101 (IO_L32N_1)
- net GND: now also U$19.108 (GND), U$19.113 (GND@1), U$19.13 (GND@2), U$19.130 (GND@3), U$19.136 (GND@4), U$19.25 (GND@5), U$19.3 (GND@6), U$19.49 (GND@7), U$19.54 (GND@8), U$19.68 (GND@9), U$19.77 (GND@10), U$19.91 (GND@11), U$19.96 (GND@12), U1.3 (GND)
- net GOUT: now also U$19.95 (IO_L40P_GCLK11_1)
- net GRAPHIC: now also U$19.137 (IO_L4N_0)
- net HSYNC: now also U$19.99 (IO_L33N_1)
- net IOINH: now also U$19.111 (IO_L66N_SCP0_0)
- net PET_VSYNC: now also U$19.92 (IO_L41N_GCLK8_1)
- net PHI2: now also J3.1 (Pin_1), U$19.126 (IO_L36N_GCLK14_0)
- net R/-W: now also U$19.124 (IO_L37P_GCLK13_0)
- net RAMA0: now also U$19.50 (IO_L31N_GCLK30_D15_2)
- net RAMA1: now also U$19.55 (IO_L30N_GCLK0_USERCCLK_2)
- net RAMA10: now also U$19.57 (IO_L14N_D12_2)
- net RAMA11: now also U$19.62 (IO_L12P_D1_MISO2_2)
- net RAMA12: now also U$19.81 (IO_L46P_1)
- net RAMA13: now also U$19.80 (IO_L46N_1)
- net RAMA14: now also U$19.83 (IO_L45P_1)
- net RAMA15: now also U$19.87 (IO_L42N_GCLK6_TRDY1_1)
- net RAMA16: now also U$19.85 (IO_L43P_GCLK5_1)
- net RAMA17: now also U$19.84 (IO_L43N_GCLK4_1)
- net RAMA18: now also U$19.88 (IO_L42P_GCLK7_1)
- net RAMA2: now also U$19.58 (IO_L14P_D11_2)
- net RAMA3: now also IC3.6 (O), U$19.60 (IO_L13P_M1_2)
- net RAMA4: now also U$19.61 (IO_L12N_D2_MISO3_2)
- net RAMA5: now also U$19.66 (IO_L2N_CMPMOSI_2)
- net RAMA6: now also U$19.75 (IO_L74P_AWAKE_1)
- net RAMA7: now also U$19.79 (IO_L47P_1)
- net RAMA8: now also U$19.78 (IO_L47N_1)
- net RAMA9: now also U$19.69 (IO_L1N_M0_CMPMISO_2)
- net RAMD0: now also U$19.47 (IO_L48N_RDRW_B_VREF_2)
- net RAMD1: now also U$19.46 (IO_L49P_D3_2)
- net RAMD2: now also U$19.39 (IO_L65P_INIT_B_2)
- net RAMD3: now also U$19.33 (IO_L2P_3)
- net RAMD4: now also U$19.34 (IO_L1N_VREF_3)
- net RAMD5: now also U$19.35 (IO_L1P_3)
- net RAMD6: now also U$19.48 (IO_L48P_D7_2)
- net RAMD7: now also U$19.51 (IO_L31P_GCLK31_D14_2)
- net RDY: now also U$19.32 (IO_L2N_3)
- net ROUT: now also U$19.97 (IO_L34N_1)
- net SPISELA/CSO_B: now also U$19.38 (IO_L65N_CSO_B_2)
- net SPISELB: now also U$19.29 (IO_L36N_3)
- net SPISELC: now also U$19.27 (IO_L37P_3)
- net SPI_ACLK: now also U$19.16 (IO_L43N_GCLK22_IRDY2_3)
- net SPI_AMOSI: now also U$19.15 (IO_L44P_GCLK21_3)
- net SPI_CLK/CCLK: now also U$19.70 (IO_L1P_CCLK_2)
- net SPI_IN3: now also U$19.67 (IO_L2P_CMPCLK_2)
- net SPI_MISO/DIN: now also U$19.65 (IO_L3P_D0_DIN_MISO_MISO1_2)
- net SPI_MOSI: now also U$19.64 (IO_L3N_MOSI_CSI_B_MISO0_2)
- net SPI_NAUDIO: now also U$19.116 (IO_L64N_SCP4_0)
- net SPI_NFLASH: now also J5.1 (Pin_1)
- net SYNC: now also U$19.121 (IO_L62P_0)
- net V12: now also U$19.128 (VCCINT), U$19.19 (VCCINT@1), U$19.28 (VCCINT@2), U$19.52 (VCCINT@3), U$19.89 (VCCINT@4)
- net V33: now also U$19.103 (VCCO_1), U$19.122 (VCCO_0), U$19.125 (VCCO_0@1), U$19.129 (VCCAUX), U$19.135 (VCCO_0@2), U$19.18 (VCCO_3@1), U$19.20 (VCCAUX@1), U$19.31 (VCCO_3), U$19.36 (VCCAUX@2), U$19.4 (VCCO_3@2), U$19.42 (VCCO_2@1), U$19.53 (VCCAUX@3), U$19.63 (VCCO_2), U$19.76 (VCCO_1@1), U$19.86 (VCCO_1@2), U$19.90 (VCCAUX@4), U1.5 (VCC)
- net VDA: now also U$19.22 (IO_L42P_GCLK25_TRDY2_3)
- net VPA: now also U$19.24 (IO_L41P_GCLK27_3)
- net VPB: now also J1.1 (Pin_1), U$19.7 (IO_L51N_3)
- net VSYNC: now also U$19.98 (IO_L34P_1)
- net at U$7.5 (TMS): now also U$19.107 (TMS)
- net at U$7.3 (TDO): now also U$19.106 (TDO)
- net at U$7.1 (TCK): now also U$19.109 (TCK)
- net at U$7.9 (TDI): now also U$19.110 (TDI)
- net M2: no longer names the net of IC3.8 (O)
- net PROG_B: no longer names the net of JP4.2, R25.1
- net PROG_B: now also U$19.37 (PROGRAM_B_2)
- net SPI_CLK renamed SPI_CLK/CCLK
- new net BE: U$1.40 (BE), U1.4
- new net IBOUT: U$19.93 (IO_L41P_GCLK9_IRDY1_1)
- new net IGOUT: U$19.74 (IO_L74N_DOUT_BUSY_1)
- new net IROUT: U$19.105 (IO_L1P_1)
- new net /BE: U$19.100 (IO_L33P_1), U1.2
Other:
- note added: "CBM-ULTIPET-V1.0A-20240330"
- note added: "For Master SPI config, M[0..1] need to be 01 (M0=1, M1=0) - doing this with '125 when DONE is low M[] are sampled when INIT_B goes high, std I/O after config DONE goes high after initialization is finished. Boot PROM connections: MOSI is SPI MOSI DIN is SPI MISO CSO_B is Boot flash /select CCLK is SPI clock (CCLK is 50 Ohm transmission line - no branches 100/100 termination)"
- note removed: "CBM-ULTIPET-V1.0A-20240104"
- note removed: "For Master SPI config, M[0..2] need to be 001 (M0=1, M1=0, M2=0) - doing this with '125 when DONE is low VS[0..2] select Flash variant M[] and VS[] are sampled when INIT_B goes high, std I/O after config DONE goes high after initialization is finished. Boot PROM connections: MOSI is SPI MOSI DIN is SPI MISO CSO_B is Boot flash /select CCLK is SPI clock (CCLK is 50 Ohm transmission line - no branc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"
- note removed: "M0"
- note removed: "VS0"
- note removed: "VS1"
- note removed: "VS2"
- moved on the sheet: IC3A, IC7A

Commit message: ultipet 1.1a board
Connections:
- net SPI_NSEL0: now reaches IC7.15 (Y0)
- net /RES: now reaches IC3.8 (O)
Other:
- note added: "1.0B: - add Pulldown from DONE to /RES to ensure proper init 1.1A: - add SPI_NSEL0 for SPI-10/UEXT connector"
- note added: "CBM-ULTIPET-V1.1A"
- note added: "CBM-ULTIPET-V1.1A-20240526"
- note removed: "CBM-ULTIPET-V1.0A"
- note removed: "CBM-ULTIPET-V1.0A-20240330"

Commit message: diverse fixes
Connections:
- net GND: now also IC3.12 (I)
- net OPENHIGH: no longer IC3.12 (I), IC3.13 (OE)
- net KEYLOCK_LED: now reaches IC3.11 (O)
- new net KEYLOCK: IC3.13 (OE)
Changed lines of the file:
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@@
 	)
 	(junction
-		(at 154.94 25.4)
-		(diameter 0)
-		(color 0 0 0 0)
-	)
-	(junction
 		(at 524.51 127)
 		(diameter 0)
@@
 		)
 	)
+	(wire
+		(pts
+			(xy 170.18 25.4) (xy 170.18 33.02)
+		)
+		(stroke
+			(width 0)
+			(type default)
+		)
+	)
 	(bus
 		(pts
@@
 	(wire
 		(pts
+			(xy 180.34 40.64) (xy 189.23 40.64)
+		)
+		(stroke
+			(width 0)
+			(type default)
+		)
+	)
+	(wire
+		(pts
 			(xy 332.74 200.66) (xy 332.74 184.15)
 		)
@@
 	(wire
 		(pts
+			(xy 160.02 40.64) (xy 157.48 40.64)
+		)
+		(stroke
+			(width 0)
+			(type default)
+		)
+	)
+	(wire
+		(pts
 			(xy 524.51 147.32) (xy 524.51 149.86)
 		)
@@
 	(wire
 		(pts
-			(xy 170.18 33.02) (xy 170.18 25.4)
-		)
-		(stroke
-			(width 0.1524)
-			(type solid)
-		)
-	)
-	(wire
-		(pts
-			(xy 160.02 40.64) (xy 154.94 40.64)
-		)
-		(stroke
-			(width 0.1524)
-			(type solid)
-		)
-	)
-	(wire
-		(pts
 			(xy 515.62 119.38) (xy 524.51 119.38)
 		)
@@
 		)
 	)
-	(wire
-		(pts
-			(xy 148.59 25.4) (xy 154.94 25.4)
-		)
-		(stroke
-			(width 0.1524)
-			(type solid)
-		)
-	)
 	(bus
 		(pts
@@
 	(wire
 		(pts
-			(xy 170.18 25.4) (xy 154.94 25.4)
-		)
-		(stroke
-			(width 0.1524)
-			(type solid)
-		)
-	)
-	(wire
-		(pts
 			(xy 185.42 269.24) (xy 185.42 289.56)
 		)
@@
 	(wire
 		(pts
-			(xy 154.94 40.64) (xy 154.94 25.4)
-		)
-		(stroke
-			(width 0.1524)
-			(type solid)
-		)
-	)
-	(wire
-		(pts
 			(xy 243.84 93.98) (xy 243.84 106.68)
 		)
@@
 	(wire
 		(pts
+			(xy 157.48 40.64) (xy 157.48 41.91)
+		)
+		(stroke
+			(width 0)
+			(type default)
+		)
+	)
+	(wire
+		(pts
 			(xy 232.41 204.47) (xy 232.41 231.14)
 		)
@@
 	(wire
 		(pts
+			(xy 157.48 25.4) (xy 170.18 25.4)
+		)
+		(stroke
+			(width 0)
+			(type default)
+		)
+	)
+	(wire
+		(pts
 			(xy 309.88 97.79) (xy 304.8 97.79)
 		)
@@
 		)
 	)
+	(global_label "KEYLOCK_LED"
+		(shape output)
+		(at 189.23 40.64 0)
+		(fields_autoplaced yes)
+		(effects
+			(font
+				(size 1.27 1.27)
+			)
+			(justify left)
+		)
+		(property "Intersheetrefs" "${INTERSHEET_REFS}"
+			(at 205.0361 40.64 0)
+			(effects
+				(font
+					(size 1.27 1.27)
+				)
+				(justify left)
+				(hide yes)
+			)
+		)
+	)
 	(global_label "RAMD1"
 		(shape bidirectional)
@@
 		)
 	)
-	(global_label "OPENHIGH"
-		(shape bidirectional)
-		(at 148.59 25.4 180)
-		(fields_autoplaced yes)
-		(effects
-			(font
-				(size 1.2446 1.2446)
-			)
-			(justify right)
-		)
-		(property "Intersheetrefs" "${INTERSHEET_REFS}"
-			(at 135.1522 25.4 0)
-			(effects
-				(font
-					(size 1.27 1.27)
-				)
-				(justify right)
-				(hide yes)
-			)
-		)
-	)
 	(global_label "RAMD5"
 		(shape bidirectional)
@@
 		)
 	)
+	(global_label "KEYLOCK"
+		(shape input)
+		(at 157.48 25.4 180)
+		(fields_autoplaced yes)
+		(effects
+			(font
+				(size 1.27 1.27)
+			)
+			(justify right)
+		)
+		(property "Intersheetrefs" "${INTERSHEET_REFS}"
+			(at 146.0886 25.4 0)
+			(effects
+				(font
+					(size 1.27 1.27)
+				)
+				(justify right)
+				(hide yes)
+			)
+		)
+	)
 	(global_label "RAMA5"
 		(shape bidirectional)
@@
 					(unit 1)
 				)
+			)
+		)
+	)
+	(symbol
+		(lib_id "cbm_ultipet_v1-eagle-import:GND")
+		(at 157.48 44.45 0)
+		(unit 1)
+		(exclude_from_sim no)
+		(in_bom yes)
+		(on_board yes)
+		(dnp no)
+		(property "Reference" "#GND0140"
+			(at 157.48 44.45 0)
+			(effects
+				(font
+					(size 1.27 1.27)
+				)
+				(hide yes)
+			)
+		)
+		(property "Value" "GND"
+			(at 154.94 46.99 0)
+			(effects
+				(font
+					(size 1.778 1.5113)
+				)
+				(justify left bottom)
+			)
+		)
+		(property "Footprint" ""
+			(at 157.48 44.45 0)
+			(effects
+				(font
+					(size 1.27 1.27)
+				)
+				(hide yes)
+			)
+		)
+		(property "Datasheet" ""
+			(at 157.48 44.45 0)
+			(effects
+				(font
+					(size 1.27 1.27)
+				)
+				(hide yes)
+			)
+		)
+		(property "Description" ""
+			(at 157.48 44.45 0)
+			(effects
+				(font
+					(size 1.27 1.27)
+				)
+				(hide yes)
+			)
+		)
+		(pin "1"
+		)
+		(instances
+			(project "cbm_ultipet_v1"
+				(path "/4dd2dd78-173f-4b46-8cce-4ed940435c94/c1121991-0565-423b-8c3b-d37496a455be"
+					(reference "#GND0140")
+					(unit 1)
+				)

Commit message: various fixes as documented in github issues
Parts:
- removed QG1: 50MHz, cbm_ultipet_v1:SG51, symbol cbm_ultipet_v1-eagle-import:CRYSTAL_RES-SG51
- removed R12: 1k5, cbm_ultipet_v1:0207_2V, symbol cbm_ultipet_v1-eagle-import:R-EU_0207/2V
- removed R5: 1k, cbm_ultipet_v1:0207_2V, symbol cbm_ultipet_v1-eagle-import:R-EU_0207/2V
- removed SJ1: SJ2W, cbm_ultipet_v1:SJ_2, symbol cbm_ultipet_v1-eagle-import:SJ2W
Connections:
- net 50MSMD is gone; now on net 50M: JS1.4 (OUT1)
Other:
- note added: "1.0B: - add Pulldown from DONE to /RES to ensure proper init 1.1A: - add SPI_NSEL0 for SPI-10/UEXT connector 1.2A: - use last gate on IC3 for shift lock LED - remove 50MHz oscillator option"
- note added: "CBM-ULTIPET-V1.2A"
- note added: "CBM-ULTIPET-V1.2A-20241013"
- note removed: "1.0B: - add Pulldown from DONE to /RES to ensure proper init 1.1A: - add SPI_NSEL0 for SPI-10/UEXT connector"
- note removed: "CBM-ULTIPET-V1.1A"
- note removed: "CBM-ULTIPET-V1.1A-20240526"
- note removed: "Voltage divider 5V to 3.3V"

Commit message: more fixes
Parts:
- IC3: value 74125D -> 74LVC125D
- IC7: value 74138D -> 74LVC138D
Changed lines of the file:
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@@
 			)
 		)
-		(property "Value" "74138D"
+		(property "Value" "74LVC138D"
 			(at 299.72 33.02 0)
 			(effects
@@
 			)
 		)
-		(property "Value" "74125D"
+		(property "Value" "74LVC125D"
 			(at 147.32 100.33 0)
 			(effects
@@
 			)
 		)
-		(property "Value" "74125D"
+		(property "Value" "74LVC125D"
 			(at 172.72 45.72 0)
 			(effects
@@
 			)
 		)
-		(property "Value" "74125D"
+		(property "Value" "74LVC125D"
 			(at 416.56 162.56 0)
 			(effects
@@
 			)
 		)
-		(property "Value" "74125D"
+		(property "Value" "74LVC125D"
 			(at 345.44 314.96 0)
 			(effects
@@
 			)
 		)
-		(property "Value" "74138D"
+		(property "Value" "74LVC138D"
 			(at 322.58 325.12 0)
 			(effects
@@
 			)
 		)
-		(property "Value" "74125D"
+		(property "Value" "74LVC125D"
 			(at 416.56 182.88 0)
 			(effects

Commit message: more work on 1.3
Parts:
- added R39, R40: 100, cbm_ultipet_v1:0207_2V, symbol cbm_ultipet_v1-eagle-import:R-EU_0207/2V
- added U9: 74LVC1G08, Package_TO_SOT_SMD:SOT-23-5, symbol 74xGxx:74LVC1G08
Connections:
- net GND: now also R40.1, U9.3 (GND)
- net SPI_CLK/CCLK: now also R39.1, R40.2, U9.1, U9.2
- net V33: now also R39.2, U9.5 (VCC)
- new net BUF_SPI_CLK: U9.4
Other:
- note added: "CCLK Line Buffer for I/O"
- note added: "CCLK Line Termination"

Commit message: work on 1.3
Parts:
- U$1: footprint cbm_ultipet_v1:PLCC44 -> Package_LCC:PLCC-44_THT-Socket
- U$19: footprint cbm_ultipet_v1:TQFP144 -> Package_QFP:TQFP-144_20x20mm_P0.5mm
Changed lines of the file:
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@@
 (kicad_sch
-	(version 20231120)
+	(version 20250114)
 	(generator "eeschema")
-	(generator_version "8.0")
+	(generator_version "9.0")
 	(paper "User" 565.963 353.212)
+	(text "TODO: why is a separate SPI clk \nneeded for FPGA and Program flash?"
+		(exclude_from_sim no)
+		(at 101.6 55.88 0)
+		(effects
+			(font
+				(size 1.27 1.27)
+			)
+			(justify left bottom)
+		)
+	)
+	(text "CPU Boot sector + boot ROM"
+		(exclude_from_sim no)
+		(at 45.72 93.98 0)
+		(effects
+			(font
+				(size 1.778 1.5113)
+			)
+			(justify left bottom)
+		)
+	)
+	(text "1.0B: \n- add Pulldown from DONE to /RES to ensure proper init\n1.1A:\n- add SPI_NSEL0 for SPI-10/UEXT connector\n1.2A:\n- use last gate on IC3 for shift lock LED\n- remove 50MHz oscillator option"
+		(exclude_from_sim no)
+		(at 406.4 279.654 0)
+		(effects
+			(font
+				(size 2.54 2.54)
+			)
+			(justify left)
+		)
+	)
+	(text "CCLK  Line\nTermination"
+		(exclude_from_sim no)
+		(at 379.984 229.87 0)
+		(effects
+			(font
+				(size 1.7 1.7)
+			)
+		)
+	)
+	(text "CBM-ULTIPET-V1.2A\n"
+		(exclude_from_sim no)
+		(at 441.96 302.26 0)
+		(effects
+			(font
+				(size 3.81 3.2385)
+			)
+			(justify left bottom)
+		)
+	)
+	(text "CBM-ULTIPET-V1.2A-20241013"
+		(exclude_from_sim no)
+		(at 441.96 325.12 0)
+		(effects
+			(font
+				(size 2.54 2.159)
+			)
+			(justify left bottom)
+		)
+	)
+	(text "CCLK  Line\nBuffer for I/O"
+		(exclude_from_sim no)
+		(at 334.264 259.334 0)
+		(effects
+			(font
+				(size 1.7 1.7)
+			)
+		)
+	)
+	(text "(C) A. Fachat"
+		(exclude_from_sim no)
+		(at 441.96 307.34 0)
+		(effects
+			(font
+				(size 2.54 2.159)
+			)
+			(justify left bottom)
+		)
+	)
+	(text "HSWAP pulldown\nduring configuration\nto enable pullups\non config+I/O pins"
+		(exclude_from_sim no)
+		(at 152.4 85.09 0)
+		(effects
+			(font
+				(size 1.778 1.5113)
+			)
+			(justify left bottom)
+		)
+	)
+	(text "For Master SPI config,\nM[0..1] need to be 01\n(M0=1, M1=0) - doing this with '125 when DONE is low\nM[] are sampled when INIT_B goes high, std I/O after config\nDONE goes high after initialization is finished.\n\nBoot PROM connections:\nMOSI is SPI MOSI\nDIN is SPI MISO\nCSO_B is Boot flash /select\nCCLK is SPI clock\n(CCLK is 50 Ohm transmission line\n- no branches 100/100 termination)"
+		(exclude_from_sim no)
+		(at 404.368 245.11 0)
+		(effects
+			(font
+				(size 1.778 1.5113)
+			)
+			(justify left bottom)
+		)
+	)
+	(text "HSWAP"
+		(exclude_from_sim no)
+		(at 198.12 77.47 90)
+		(effects
+			(font
+				(size 1.778 1.5113)
+			)
+			(justify left bottom)
+		)
+	)
+	(text "FPGA Configuration Flash ROM"
+		(exclude_from_sim no)
+		(at 43.18 22.86 0)
+		(effects
+			(font
+				(size 1.778 1.5113)
+			)
+			(justify left bottom)
+		)
+	)
 	(junction
 		(at 524.51 116.84)
@@
 		)
 	)
-	(text "TODO: why is a separate SPI clk \nneeded for FPGA and Program flash?"
-		(exclude_from_sim no)
-		(at 101.6 55.88 0)
-		(effects
-			(font
-				(size 1.27 1.27)
-			)
-			(justify left bottom)
-		)
-	)
-	(text "CPU Boot sector + boot ROM"
-		(exclude_from_sim no)
-		(at 45.72 93.98 0)
-		(effects
-			(font
-				(size 1.778 1.5113)
-			)
-			(justify left bottom)
-		)
-	)
-	(text "1.0B: \n- add Pulldown from DONE to /RES to ensure proper init\n1.1A:\n- add SPI_NSEL0 for SPI-10/UEXT connector\n1.2A:\n- use last gate on IC3 for shift lock LED\n- remove 50MHz oscillator option"
-		(exclude_from_sim no)
-		(at 406.4 279.654 0)
-		(effects
-			(font
-				(size 2.54 2.54)
-			)
-			(justify left)
-		)
-	)
-	(text "CCLK  Line\nTermination"
-		(exclude_from_sim no)
-		(at 379.984 229.87 0)
-		(effects
-			(font
-				(size 1.7 1.7)
-			)
-		)
-	)
-	(text "CBM-ULTIPET-V1.2A\n"
-		(exclude_from_sim no)
-		(at 441.96 302.26 0)
-		(effects
-			(font
-				(size 3.81 3.2385)
-			)
-			(justify left bottom)
-		)
-	)
-	(text "CBM-ULTIPET-V1.2A-20241013"
-		(exclude_from_sim no)
-		(at 441.96 325.12 0)
-		(effects
-			(font
-				(size 2.54 2.159)
-			)
-			(justify left bottom)
-		)
-	)
-	(text "CCLK  Line\nBuffer for I/O"
-		(exclude_from_sim no)
-		(at 334.264 259.334 0)
-		(effects
-			(font
-				(size 1.7 1.7)
-			)
-		)
-	)
-	(text "(C) A. Fachat"
-		(exclude_from_sim no)
-		(at 441.96 307.34 0)
-		(effects
-			(font
-				(size 2.54 2.159)
-			)
-			(justify left bottom)
-		)
-	)
-	(text "HSWAP pulldown\nduring configuration\nto enable pullups\non config+I/O pins"
-		(exclude_from_sim no)
-		(at 152.4 85.09 0)
-		(effects
-			(font
-				(size 1.778 1.5113)
-			)
-			(justify left bottom)
-		)
-	)
-	(text "For Master SPI config,\nM[0..1] need to be 01\n(M0=1, M1=0) - doing this with '125 when DONE is low\nM[] are sampled when INIT_B goes high, std I/O after config\nDONE goes high after initialization is finished.\n\nBoot PROM connections:\nMOSI is SPI MOSI\nDIN is SPI MISO\nCSO_B is Boot flash /select\nCCLK is SPI clock\n(CCLK is 50 Ohm transmission line\n- no branches 100/100 termination)"
-		(exclude_from_sim no)
-		(at 404.368 245.11 0)
-		(effects
-			(font
-				(size 1.778 1.5113)
-			)
-			(justify left bottom)
-		)
-	)
-	(text "HSWAP"
-		(exclude_from_sim no)
-		(at 198.12 77.47 90)
-		(effects
-			(font
-				(size 1.778 1.5113)
-			)
-			(justify left bottom)
-		)
-	)
-	(text "FPGA Configuration Flash ROM"
-		(exclude_from_sim no)
-		(at 43.18 22.86 0)
-		(effects
-			(font
-				(size 1.778 1.5113)
-			)
-			(justify left bottom)
-		)
-	)
 	(label "VDA"
 		(at 247.65 213.36 90)
@@
 			)
 		)
-		(property "Footprint" "cbm_ultipet_v1:TQFP144"
+		(property "Footprint" "Package_QFP:TQFP-144_20x20mm_P0.5mm"
 			(at 485.14 187.96 0)
 			(effects
@@
 			)
 		)
-		(property "Footprint" "cbm_ultipet_v1:TQFP144"
+		(property "Footprint" "Package_QFP:TQFP-144_20x20mm_P0.5mm"
 			(at 284.48 148.59 0)
 			(effects
@@
 			)
 		)
-		(property "Footprint" "cbm_ultipet_v1:PLCC44"
+		(property "Footprint" "Package_LCC:PLCC-44_THT-Socket"
 			(at 160.02 259.08 0)
 			(effects
@@
 			)
 		)
-		(property "Footprint" "cbm_ultipet_v1:PLCC44"
+		(property "Footprint" "Package_LCC:PLCC-44_THT-Socket"
 			(at 508 205.74 0)
 			(effects
@@
 			)
 		)
-		(property "Footprint" "cbm_ultipet_v1:PLCC44"
+		(property "Footprint" "Package_LCC:PLCC-44_THT-Socket"
 			(at 518.16 213.36 0)
 			(effects
@@
 			)
 		)
-		(property "Footprint" "cbm_ultipet_v1:TQFP144"
+		(property "Footprint" "Package_QFP:TQFP-144_20x20mm_P0.5mm"
 			(at 482.6 111.76 0)
 			(effects
