File: Board/CPU,_FPGA,_FRAM.kicad_sch (KiCad schematic)
At the start: 25 parts, among them IC1 RAMSOCK32TO512KSOP, IC3 74LVC125D, IC7 74LVC138D, J1 Conn_01x01_Pin, J3 Conn_01x01_Pin, J4 Conn_01x01_Pin, J5 Conn_01x01_Pin, U1 74LVC1G04, U9 74LVC1G08

Commit message: work on r1.3
Parts:
- U$18, U$4: footprint cbm_ultipet_v1:DIL08 -> Package_DIP:DIP-8_W7.62mm_Socket_LongPads
Changed lines of the file:
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@@
 			)
 		)
-		(property "Footprint" "cbm_ultipet_v1:DIL08"
+		(property "Footprint" "Package_DIP:DIP-8_W7.62mm_Socket_LongPads"
 			(at 60.96 38.1 0)
 			(effects
@@
 			)
 		)
-		(property "Footprint" "cbm_ultipet_v1:DIL08"
+		(property "Footprint" "Package_DIP:DIP-8_W7.62mm_Socket_LongPads"
 			(at 60.96 73.66 0)
 			(effects

Commit message: more work on r1.3
Connections:
- net /BE_DOUT: now also U$19.99 (IO_L33N_1); no longer U$19.133 (IO_L34N_GCLK18_0)
- net /BE_OUT: now also U$19.98 (IO_L34P_1); no longer U$19.132 (IO_L35P_GCLK17_0)
- net /FRAMSEL: now also U$19.127 (IO_L36P_GCLK15_0); no longer U$19.120 (IO_L62N_VREF_0)
- net /MEMSEL: now also U$19.101 (IO_L32N_1); no longer U$19.112 (IO_L66P_SCP1_0)
- net /RAMWE: now also U$19.81 (IO_L46P_1); no longer U$19.82 (IO_L45N_1)
- net /RES: now also U$19.94 (IO_L40N_GCLK10_1); no longer U$19.117 (IO_L64P_SCP5_0)
- net A12: now also U$19.132 (IO_L35P_GCLK17_0); no longer U$19.127 (IO_L36P_GCLK15_0)
- net A14: now also U$19.131 (IO_L35N_GCLK16_0); no longer U$19.119 (IO_L63P_SCP7_0)
- net A15: now also U$19.133 (IO_L34N_GCLK18_0); no longer U$19.131 (IO_L35N_GCLK16_0)
- net BE_IN: now also U$19.97 (IO_L34N_1); no longer U$19.118 (IO_L63N_SCP6_0)
- net BOUT: now also U$19.116 (IO_L64N_SCP4_0); no longer U$19.94 (IO_L40N_GCLK10_1)
- net CPHI2: now also U$19.105 (IO_L1P_1); no longer U$19.114 (IO_L65N_SCP2_0)
- net EXTIO: now also U$19.93 (IO_L41P_GCLK9_IRDY1_1); no longer U$19.115 (IO_L65P_SCP3_0)
- net FA19: now also U$19.112 (IO_L66P_SCP1_0); no longer U$19.101 (IO_L32N_1)
- net GOUT: now also U$19.118 (IO_L63N_SCP6_0); no longer U$19.95 (IO_L40P_GCLK11_1)
- net HSYNC: now also U$19.114 (IO_L65N_SCP2_0); no longer U$19.99 (IO_L33N_1)
- net IBOUT: now also U$19.117 (IO_L64P_SCP5_0); no longer U$19.93 (IO_L41P_GCLK9_IRDY1_1)
- net IGOUT: now also U$19.119 (IO_L63P_SCP7_0); no longer U$19.74 (IO_L74N_DOUT_BUSY_1)
- net IROUT: now also U$19.121 (IO_L62P_0); no longer U$19.105 (IO_L1P_1)
- net PET_VSYNC: now also U$19.88 (IO_L42P_GCLK7_1); no longer U$19.92 (IO_L41N_GCLK8_1)
- net RAMA12: now also U$19.80 (IO_L46N_1); no longer U$19.81 (IO_L46P_1)
- net RAMA13: now also U$19.79 (IO_L47P_1); no longer U$19.80 (IO_L46N_1)
- net RAMA14: now also U$19.82 (IO_L45N_1); no longer U$19.83 (IO_L45P_1)
- net RAMA15: now also U$19.85 (IO_L43P_GCLK5_1); no longer U$19.87 (IO_L42N_GCLK6_TRDY1_1)
- net RAMA16: now also U$19.84 (IO_L43N_GCLK4_1); no longer U$19.85 (IO_L43P_GCLK5_1)
- net RAMA17: now also U$19.83 (IO_L45P_1); no longer U$19.84 (IO_L43N_GCLK4_1)
- net RAMA18: now also U$19.87 (IO_L42N_GCLK6_TRDY1_1); no longer U$19.88 (IO_L42P_GCLK7_1)
- net RAMA6: now also U$19.74 (IO_L74N_DOUT_BUSY_1); no longer U$19.75 (IO_L74P_AWAKE_1)
- net RAMA7: now also U$19.78 (IO_L47N_1); no longer U$19.79 (IO_L47P_1)
- net RAMA8: now also U$19.75 (IO_L74P_AWAKE_1); no longer U$19.78 (IO_L47N_1)
- net ROUT: now also U$19.120 (IO_L62N_VREF_0); no longer U$19.97 (IO_L34N_1)
- net SPI_NAUDIO: now also U$19.92 (IO_L41N_GCLK8_1); no longer U$19.116 (IO_L64N_SCP4_0)
- net SYNC: now also U$19.95 (IO_L40P_GCLK11_1); no longer U$19.121 (IO_L62P_0)
- net VSYNC: now also U$19.115 (IO_L65P_SCP3_0); no longer U$19.98 (IO_L34P_1)
Other:
- note added: "1.0B: - add Pulldown from DONE to /RES to ensure proper init 1.1A: - add SPI_NSEL0 for SPI-10/UEXT connector 1.2A: - use last gate on IC3 for shift lock LED - remove 50MHz oscillator option 1.3A: - move (I)RGB out to N/P pair driver pins to prep for HDMI"
- note added: "CBM-ULTIPET-V1.3A"
- note added: "CBM-ULTIPET-V1.3A-20250806"
- note removed: "1.0B: - add Pulldown from DONE to /RES to ensure proper init 1.1A: - add SPI_NSEL0 for SPI-10/UEXT connector 1.2A: - use last gate on IC3 for shift lock LED - remove 50MHz oscillator option"
- note removed: "CBM-ULTIPET-V1.2A"
- note removed: "CBM-ULTIPET-V1.2A-20241013"

Commit message: layout work on r1.3a
Parts:
- removed IC1: RAMSOCK32TO512KSOP, cbm_ultipet_v1:SOP32, symbol cbm_ultipet_v1-eagle-import:RAMSOCK32TO512KSOP
- added C166, C167: 0.1u, Capacitor_SMD:C_0603_1608Metric, symbol Device:C_Small
- added IC1: 512k x8 10ns SRAM, Package_SO:TSOP-II-44_10.16x18.41mm_P0.8mm, symbol Memory_RAM:IS61C5128AL-10TLI
Connections:
- net /RAMCS/M1 is gone; now on net RAMA14: U$19.59 (IO_L13N_D10_2)
- net /RAMWE: now also U$19.74 (IO_L74N_DOUT_BUSY_1); no longer U$19.81 (IO_L46P_1)
- net A0: now also IC1.3 (A0)
- net A1: now also U$19.41 (IO_L64P_D8_2), IC1.4 (A1); no longer U$19.56 (IO_L30P_GCLK1_D13_2)
- net A10: now also IC1.26 (A10)
- net A11: now also IC1.27 (A11)
- net A12: now also IC1.28 (A12)
- net A13: now also IC1.29 (A13)
- net A14: now also IC1.30 (A14)
- net A2: now also U$19.33 (IO_L2P_3), IC1.5 (A2); no longer U$19.45 (IO_L49N_D4_2)
- net A3: now also U$19.39 (IO_L65P_INIT_B_2), IC1.6 (A3); no longer U$19.43 (IO_L62N_D6_2)
- net A4: now also U$19.34 (IO_L1N_VREF_3), IC1.7 (A4); no longer U$19.44 (IO_L62P_D5_2)
- net A5: now also IC1.16 (A5)
- net A6: now also U$19.35 (IO_L1P_3), IC1.17 (A6); no longer U$19.41 (IO_L64P_D8_2)
- net A7: now also IC1.18 (A7)
- net A8: now also IC1.19 (A8)
- net A9: now also IC1.20 (A9)
- net D0: now also IC1.9 (I/O0)
- net D1: now also IC1.10 (I/O1)
- net D2: now also IC1.13 (I/O2)
- net D3: now also IC1.14 (I/O3)
- net D4: now also IC1.31 (I/O4)
- net D5: now also IC1.32 (I/O5)
- net D6: now also IC1.35 (I/O6)
- net D7: now also IC1.36 (I/O7)
- net FA15: now also IC1.38 (A15)
- net FA16: now also IC1.39 (A16)
- net FA17: now also IC1.40 (A17)
- net FA18: now also IC1.41 (A18)
- net GND: now also C166.2, C167.2, IC1.12 (GND), IC1.34 (GND)
- net R/-W: now also IC1.15 (~{WE})
- net RAMA0: now also U$19.87 (IO_L42N_GCLK6_TRDY1_1); no longer U$19.50 (IO_L31N_GCLK30_D15_2)
- net RAMA1: now also U$19.85 (IO_L43P_GCLK5_1); no longer U$19.55 (IO_L30N_GCLK0_USERCCLK_2)
- net RAMA10: now also U$19.55 (IO_L30N_GCLK0_USERCCLK_2); no longer U$19.57 (IO_L14N_D12_2)
- net RAMA11: now also U$19.56 (IO_L30P_GCLK1_D13_2); no longer U$19.62 (IO_L12P_D1_MISO2_2)
- net RAMA12: now also U$19.57 (IO_L14N_D12_2); no longer U$19.80 (IO_L46N_1)
- net RAMA13: now also U$19.58 (IO_L14P_D11_2); no longer U$19.79 (IO_L47P_1)
- net RAMA14: no longer U$19.82 (IO_L45N_1)
- net RAMA15: now also U$19.46 (IO_L49P_D3_2); no longer U$19.85 (IO_L43P_GCLK5_1)
- net RAMA16: now also U$19.45 (IO_L49N_D4_2); no longer U$19.84 (IO_L43N_GCLK4_1)
- net RAMA17: now also U$19.44 (IO_L62P_D5_2); no longer U$19.83 (IO_L45P_1)
- net RAMA18: now also U$19.43 (IO_L62N_D6_2); no longer U$19.87 (IO_L42N_GCLK6_TRDY1_1)
- net RAMA2: now also U$19.84 (IO_L43N_GCLK4_1); no longer U$19.58 (IO_L14P_D11_2)
- net RAMA3: now also U$19.83 (IO_L45P_1); no longer IC3.6 (O), U$19.60 (IO_L13P_M1_2)
- net RAMA4: now also U$19.82 (IO_L45N_1); no longer U$19.61 (IO_L12N_D2_MISO3_2)
- net RAMA5: now also IC3.6 (O), U$19.60 (IO_L13P_M1_2); no longer U$19.66 (IO_L2N_CMPMOSI_2)
- net RAMA6: now also U$19.61 (IO_L12N_D2_MISO3_2); no longer U$19.74 (IO_L74N_DOUT_BUSY_1)
- net RAMA7: now also U$19.62 (IO_L12P_D1_MISO2_2); no longer U$19.78 (IO_L47N_1)
- net RAMA8: now also U$19.66 (IO_L2N_CMPMOSI_2); no longer U$19.75 (IO_L74P_AWAKE_1)
- net RAMD0: now also U$19.80 (IO_L46N_1); no longer U$19.47 (IO_L48N_RDRW_B_VREF_2)
- net RAMD1: now also U$19.79 (IO_L47P_1); no longer U$19.46 (IO_L49P_D3_2)
- net RAMD2: now also U$19.78 (IO_L47N_1); no longer U$19.39 (IO_L65P_INIT_B_2)
- net RAMD3: now also U$19.75 (IO_L74P_AWAKE_1); no longer U$19.33 (IO_L2P_3)
- net RAMD4: now also U$19.51 (IO_L31P_GCLK31_D14_2); no longer U$19.34 (IO_L1N_VREF_3)
- net RAMD5: now also U$19.50 (IO_L31N_GCLK30_D15_2); no longer U$19.35 (IO_L1P_3)
- net RAMD7: now also U$19.47 (IO_L48N_RDRW_B_VREF_2); no longer U$19.51 (IO_L31P_GCLK31_D14_2)
- net V33: now also C166.1, C167.1, IC1.11 (VDD), IC1.33 (VDD)
- new net /FRAMSEL: IC1.37 (~{OE}), IC1.8 (~{CE})
- new net /RAMCS: U$19.81 (IO_L46P_1)
Other:
- note added: "1.0B: - add Pulldown from DONE to /RES to ensure proper init 1.1A: - add SPI_NSEL0 for SPI-10/UEXT connector 1.2A: - use last gate on IC3 for shift lock LED - remove 50MHz oscillator option 1.3A: - move (I)RGB out to N/P pair driver pins to prep for HDMI - replace 5V SRAM with 3.3V type"
- note removed: "1.0B: - add Pulldown from DONE to /RES to ensure proper init 1.1A: - add SPI_NSEL0 for SPI-10/UEXT connector 1.2A: - use last gate on IC3 for shift lock LED - remove 50MHz oscillator option 1.3A: - move (I)RGB out to N/P pair driver pins to prep for HDMI"
- moved on the sheet: IC3E, IC7B

Commit message: more layout work on r1.3
Parts:
- removed JS1: RENOSCXLH, cbm_ultipet_v1:RENJS6, symbol cbm_ultipet_v1-eagle-import:RENOSCXLH
- removed R30: 10k, cbm_ultipet_v1:0207_2V, symbol cbm_ultipet_v1-eagle-import:R-EU_0207/2V
- added R47: 10k, Resistor_SMD:R_0805_2012Metric_Pad1.20x1.40mm_HandSolder, symbol csa_ultracpu-eagle-import:R-EU_0207/2V
- added X1: SG-8002CE, Oscillator:Oscillator_SMD_SeikoEpson_SG8002CE-4Pin_3.2x2.5mm, symbol Oscillator:SG-8002CE
Connections:
- net 50M: now also X1.3 (OUT)
- net GND: now also X1.2 (GND)
- net V33: now also R47.1, X1.4 (Vcc)
- new net: R47.2, X1.1 (OE)
Other:
- note added: "1.0B: - add Pulldown from DONE to /RES to ensure proper init 1.1A: - add SPI_NSEL0 for SPI-10/UEXT connector 1.2A: - use last gate on IC3 for shift lock LED - remove 50MHz oscillator option 1.3A: - move (I)RGB out to N/P pair driver pins to prep for HDMI - replace 5V SRAM with 3.3V type - different footprint for clock oscillator"
- note removed: "1.0B: - add Pulldown from DONE to /RES to ensure proper init 1.1A: - add SPI_NSEL0 for SPI-10/UEXT connector 1.2A: - use last gate on IC3 for shift lock LED - remove 50MHz oscillator option 1.3A: - move (I)RGB out to N/P pair driver pins to prep for HDMI - replace 5V SRAM with 3.3V type"

Commit message: rename U refs to UX*
Parts:
- renumbered U$1 to UX1, U$18 to UX18, U$19 to UX19, U$4 to UX4, U$7 to UX7
Changed lines of the file:
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@@
 		(on_board yes)
 		(dnp no)
-		(property "Reference" "U$18"
+		(property "Reference" "UX18"
 			(at 55.88 27.94 0)
 			(effects
@@
 			(project "cbm_ultipet_v1"
 				(path "/4dd2dd78-173f-4b46-8cce-4ed940435c94/c1121991-0565-423b-8c3b-d37496a455be"
-					(reference "U$18")
+					(reference "UX18")
 					(unit 1)
 				)
@@
 		(on_board yes)
 		(dnp no)
-		(property "Reference" "U$19"
+		(property "Reference" "UX19"
 			(at 480.06 179.07 0)
 			(effects
@@
 			(project "cbm_ultipet_v1"
 				(path "/4dd2dd78-173f-4b46-8cce-4ed940435c94/c1121991-0565-423b-8c3b-d37496a455be"
-					(reference "U$19")
+					(reference "UX19")
 					(unit 3)
 				)
@@
 		(on_board yes)
 		(dnp no)
-		(property "Reference" "U$19"
+		(property "Reference" "UX19"
 			(at 275.59 153.67 0)
 			(effects
@@
 			(project "cbm_ultipet_v1"
 				(path "/4dd2dd78-173f-4b46-8cce-4ed940435c94/c1121991-0565-423b-8c3b-d37496a455be"
-					(reference "U$19")
+					(reference "UX19")
 					(unit 1)
 				)
@@
 		(on_board yes)
 		(dnp no)
-		(property "Reference" "U$1"
+		(property "Reference" "UX1"
 			(at 141.605 247.015 0)
 			(effects
@@
 			(project "cbm_ultipet_v1"
 				(path "/4dd2dd78-173f-4b46-8cce-4ed940435c94/c1121991-0565-423b-8c3b-d37496a455be"
-					(reference "U$1")
+					(reference "UX1")
 					(unit 1)
 				)
@@
 		(on_board yes)
 		(dnp no)
-		(property "Reference" "U$7"
+		(property "Reference" "UX7"
 			(at 367.665 50.165 0)
 			(effects
@@
 			(project "cbm_ultipet_v1"
 				(path "/4dd2dd78-173f-4b46-8cce-4ed940435c94/c1121991-0565-423b-8c3b-d37496a455be"
-					(reference "U$7")
+					(reference "UX7")
 					(unit 2)
 				)
@@
 		(on_board yes)
 		(dnp no)
-		(property "Reference" "U$4"
+		(property "Reference" "UX4"
 			(at 55.88 63.5 0)
 			(effects
@@
 			(project "cbm_ultipet_v1"
 				(path "/4dd2dd78-173f-4b46-8cce-4ed940435c94/c1121991-0565-423b-8c3b-d37496a455be"
-					(reference "U$4")
+					(reference "UX4")
 					(unit 1)
 				)
@@
 		(on_board yes)
 		(dnp no)
-		(property "Reference" "U$1"
+		(property "Reference" "UX1"
 			(at 499.745 193.675 0)
 			(effects
@@
 			(project "cbm_ultipet_v1"
 				(path "/4dd2dd78-173f-4b46-8cce-4ed940435c94/c1121991-0565-423b-8c3b-d37496a455be"
-					(reference "U$1")
+					(reference "UX1")
 					(unit 3)
 				)
@@
 		(on_board yes)
 		(dnp no)
-		(property "Reference" "U$7"
+		(property "Reference" "UX7"
 			(at 466.725 201.295 0)
 			(effects
@@
 			(project "cbm_ultipet_v1"
 				(path "/4dd2dd78-173f-4b46-8cce-4ed940435c94/c1121991-0565-423b-8c3b-d37496a455be"
-					(reference "U$7")
+					(reference "UX7")
 					(unit 1)
 				)
@@
 		(on_board yes)
 		(dnp no)
-		(property "Reference" "U$1"
+		(property "Reference" "UX1"
 			(at 509.905 201.295 0)
 			(effects
@@
 			(project "cbm_ultipet_v1"
 				(path "/4dd2dd78-173f-4b46-8cce-4ed940435c94/c1121991-0565-423b-8c3b-d37496a455be"
-					(reference "U$1")
+					(reference "UX1")
 					(unit 2)
 				)
@@
 		(on_board yes)
 		(dnp no)
-		(property "Reference" "U$19"
+		(property "Reference" "UX19"
 			(at 477.52 102.87 0)
 			(effects
@@
 			(project "cbm_ultipet_v1"
 				(path "/4dd2dd78-173f-4b46-8cce-4ed940435c94/c1121991-0565-423b-8c3b-d37496a455be"
-					(reference "U$19")
+					(reference "UX19")
 					(unit 2)
 				)
@@
 		(on_board yes)
 		(dnp no)
-		(property "Reference" "U$7"
+		(property "Reference" "UX7"
 			(at 362.585 45.085 0)
 			(effects
@@
 			(project "cbm_ultipet_v1"
 				(path "/4dd2dd78-173f-4b46-8cce-4ed940435c94/c1121991-0565-423b-8c3b-d37496a455be"
-					(reference "U$7")
+					(reference "UX7")
 					(unit 3)
 				)

Commit message: add C64 restore
Other:
- moved on the sheet: J3, J4
