File: Board/cbm_ultipet_v1.kicad_sch (KiCad schematic)
At the start: 0 parts

Commit message: ultipet 1.1a board
Other:
- sheet NANO488 renamed I2C,UEXT
- sheet I2C,UEXT: file NANO488.kicad_sch -> I2C,UEXT.kicad_sch
Changed lines of the file:
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@@
 			(color 0 0 0 0.0000)
 		)
-		(property "Sheetname" "NANO488"
+		(property "Sheetname" "I2C,UEXT"
 			(at 25.4 177.0884 0)
 			(effects
@@
 			)
 		)
-		(property "Sheetfile" "NANO488.kicad_sch"
+		(property "Sheetfile" "I2C,UEXT.kicad_sch"
 			(at 25.4 182.1946 0)
 			(effects
