File: Board/SID.kicad_sch (KiCad schematic)
At the start: 24 parts, among them IC25 74139N

Commit message: Ultipet 1.0A final
Parts:
- added JP1: JP1E, cbm_ultipet_v1:JP1, symbol cbm_ultipet_v1-eagle-import:JP1E
Connections:
- net SIDLEFT: now also JP1.1
- net SIDRIGHT: now also JP1.2
Other:
- note added: "Absolutely only connect if only a single SID is populated on the board!!!"
- note added: "CBM-ULTIPET-1.0A-20240331"
- note added: "SID 1"
- note added: "SID 2"
- note removed: "CBM-ULTIPET-1.0A-20240104"

Commit message: ultipet 1.1a board
Other:
- note added: "CBM-ULTIPET-V1.1A"
- note removed: "CBM-ULTIPET-V1.0A"
Changed lines of the file:
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@@
 		)
 	)
-	(text "CBM-ULTIPET-V1.0A"
+	(text "CBM-ULTIPET-V1.1A\n"
 		(exclude_from_sim no)
 		(at 340.36 198.12 0)

Commit message: update SID footprints - still conflicting
Parts:
- U$22: footprint cbm_ultipet_v1:DIL28 -> cbm_ultipet_v1:SID_FPGASID
- U$23: footprint cbm_ultipet_v1:DIL28 -> cbm_ultipet_v1:SID_XSID
Changed lines of the file:
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@@
 			)
 		)
-		(property "Footprint" "cbm_ultipet_v1:DIL28"
+		(property "Footprint" "cbm_ultipet_v1:SID_XSID"
 			(at 223.52 180.34 0)
 			(effects
@@
 			)
 		)
-		(property "Footprint" "cbm_ultipet_v1:DIL28"
+		(property "Footprint" "cbm_ultipet_v1:SID_FPGASID"
 			(at 223.52 114.3 0)
 			(effects

Commit message: various fixes as documented in github issues
Parts:
- removed C75: 100n, cbm_ultipet_v1:C025-025X050, symbol cbm_ultipet_v1-eagle-import:C-EU025-025X050
Other:
- note added: "Locate next to each other so DAC could be fed into extin"
Changed lines of the file:
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@@
 	)
 	(junction
-		(at 66.04 40.64)
-		(diameter 0)
-		(color 0 0 0 0)
-	)
-	(junction
 		(at 76.2 40.64)
 		(diameter 0)
@@
 		(color 0 0 0 0)
 	)
-	(junction
-		(at 66.04 27.94)
-		(diameter 0)
-		(color 0 0 0 0)
-	)
 	(bus_entry
 		(at 190.5 177.8)
@@
 	(wire
 		(pts
-			(xy 66.04 40.64) (xy 66.04 38.1)
-		)
-		(stroke
-			(width 0.1524)
-			(type solid)
-		)
-	)
-	(wire
-		(pts
 			(xy 314.96 195.58) (xy 317.5 195.58)
 		)
@@
 	(wire
 		(pts
-			(xy 66.04 27.94) (xy 76.2 27.94)
-		)
-		(stroke
-			(width 0.1524)
-			(type solid)
-		)
-	)
-	(wire
-		(pts
-			(xy 66.04 30.48) (xy 66.04 27.94)
+			(xy 55.88 27.94) (xy 76.2 27.94)
 		)
 		(stroke
@@
 	(wire
 		(pts
-			(xy 55.88 27.94) (xy 66.04 27.94)
-		)
-		(stroke
-			(width 0.1524)
-			(type solid)
-		)
-	)
-	(wire
-		(pts
 			(xy 243.84 137.16) (xy 254 137.16)
 		)
@@
 	(wire
 		(pts
-			(xy 55.88 40.64) (xy 66.04 40.64)
-		)
-		(stroke
-			(width 0.1524)
-			(type solid)
-		)
-	)
-	(wire
-		(pts
 			(xy 86.36 30.48) (xy 86.36 27.94)
 		)
@@
 	(wire
 		(pts
-			(xy 66.04 40.64) (xy 76.2 40.64)
+			(xy 55.88 40.64) (xy 76.2 40.64)
 		)
 		(stroke
@@
 		)
 	)
+	(text "Locate next to each other so\nDAC could be fed into extin"
+		(exclude_from_sim no)
+		(at 266.446 38.608 0)
+		(effects
+			(font
+				(size 1.27 1.27)
+			)
+		)
+	)
 	(text "$E86x-$E87x"
 		(exclude_from_sim no)
@@
 					(unit 1)
 				)
-			)
-		)
-	)
-	(symbol
-		(lib_id "cbm_ultipet_v1-eagle-import:C-EU025-025X050")
-		(at 66.04 33.02 0)
-		(unit 1)
-		(exclude_from_sim no)
-		(in_bom yes)
-		(on_board yes)
-		(dnp no)
-		(property "Reference" "C75"
-			(at 67.564 32.639 0)
-			(effects
-				(font
-					(size 1.778 1.5113)
-				)
-				(justify left bottom)
-			)
-		)
-		(property "Value" "100n"
-			(at 67.564 37.719 0)
-			(effects
-				(font
-					(size 1.778 1.5113)
-				)
-				(justify left bottom)
-			)
-		)
-		(property "Footprint" "cbm_ultipet_v1:C025-025X050"
-			(at 66.04 33.02 0)
-			(effects
-				(font
-					(size 1.27 1.27)
-				)
-				(hide yes)
-			)
-		)
-		(property "Datasheet" ""
-			(at 66.04 33.02 0)
-			(effects
-				(font
-					(size 1.27 1.27)
-				)
-				(hide yes)
-			)
-		)
-		(property "Description" ""
-			(at 66.04 33.02 0)
-			(effects
-				(font
-					(size 1.27 1.27)
-				)
-				(hide yes)
-			)
-		)
-		(pin "2"
-		)
-		(pin "1"
-		)
-		(instances
-			(project "cbm_ultipet_v1"
-				(path "/4dd2dd78-173f-4b46-8cce-4ed940435c94/ef987787-576d-4ba9-8915-c171f881d1b8"
-					(reference "C75")
-					(unit 1)
-				)

Commit message: replace some ultipet specific TQFP with easier to solder parts
Parts:
- U$22: footprint cbm_ultipet_v1:SID_FPGASID -> cbm_ultipet_v1:DIL28
- U$23: footprint cbm_ultipet_v1:SID_XSID -> cbm_ultipet_v1:DIL28
Changed lines of the file:
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@@
 			)
 		)
-		(property "Footprint" "cbm_ultipet_v1:SID_XSID"
+		(property "Footprint" "cbm_ultipet_v1:DIL28"
 			(at 223.52 180.34 0)
 			(effects
@@
 			)
 		)
-		(property "Footprint" "cbm_ultipet_v1:SID_FPGASID"
+		(property "Footprint" "cbm_ultipet_v1:DIL28"
 			(at 223.52 114.3 0)
 			(effects

Commit message: more work on 1.3
Parts:
- added J9: Conn_01x01_Pin, Connector_PinHeader_2.54mm:PinHeader_1x01_P2.54mm_Vertical, symbol Connector:Conn_01x01_Pin
Connections:
- net at IC25.5 (Y1), U$23.8 (/CS): now also J9.1 (Pin_1)
Other:
- note added: "SID2 /CS for FPGASID with Dual SIDs in SID1 socket"
Changed lines of the file:
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@@
 	)
 	(junction
+		(at 172.72 170.18)
+		(diameter 0)
+		(color 0 0 0 0)
+	)
+	(junction
 		(at 314.96 149.86)
 		(diameter 0)
@@
 	(wire
 		(pts
+			(xy 154.94 179.07) (xy 172.72 179.07)
+		)
+		(stroke
+			(width 0)
+			(type default)
+		)
+	)
+	(wire
+		(pts
 			(xy 264.16 53.34) (xy 264.16 66.04)
 		)
@@
 		)
 	)
+	(wire
+		(pts
+			(xy 172.72 179.07) (xy 172.72 170.18)
+		)
+		(stroke
+			(width 0)
+			(type default)
+		)
+	)
 	(bus
 		(pts
@@
 		)
 	)
+	(text "SID2 /CS for \nFPGASID with\nDual SIDs in SID1\nsocket"
+		(exclude_from_sim no)
+		(at 153.162 185.674 0)
+		(effects
+			(font
+				(size 1.27 1.27)
+			)
+		)
+	)
 	(text "CBM-ULTIPET-V1.1A\n"
 		(exclude_from_sim no)
@@
 					(unit 1)
 				)
+			)
+		)
+	)
+	(symbol
+		(lib_id "Connector:Conn_01x01_Pin")
+		(at 149.86 179.07 0)
+		(unit 1)
+		(exclude_from_sim no)
+		(in_bom yes)
+		(on_board yes)
+		(dnp no)
+		(fields_autoplaced yes)
+		(property "Reference" "J9"
+			(at 150.495 173.99 0)
+			(effects
+				(font
+					(size 1.27 1.27)
+				)
+			)
+		)
+		(property "Value" "Conn_01x01_Pin"
+			(at 150.495 176.53 0)
+			(effects
+				(font
+					(size 1.27 1.27)
+				)
+			)
+		)
+		(property "Footprint" "Connector_PinHeader_2.54mm:PinHeader_1x01_P2.54mm_Vertical"
+			(at 149.86 179.07 0)
+			(effects
+				(font
+					(size 1.27 1.27)
+				)
+				(hide yes)
+			)
+		)
+		(property "Datasheet" "~"
+			(at 149.86 179.07 0)
+			(effects
+				(font
+					(size 1.27 1.27)
+				)
+				(hide yes)
+			)
+		)
+		(property "Description" "Generic connector, single row, 01x01, script generated"
+			(at 149.86 179.07 0)
+			(effects
+				(font
+					(size 1.27 1.27)
+				)
+				(hide yes)
+			)
+		)
+		(pin "1"
+		)
+		(instances
+			(project ""
+				(path "/4dd2dd78-173f-4b46-8cce-4ed940435c94/ef987787-576d-4ba9-8915-c171f881d1b8"
+					(reference "J9")
+					(unit 1)
+				)

Commit message: work on 1.3
Parts:
- IC25: footprint cbm_ultipet_v1:DIL16 -> Package_DIP:DIP-16_W7.62mm_Socket_LongPads
Changed lines of the file:
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@@
 (kicad_sch
-	(version 20231120)
+	(version 20250114)
 	(generator "eeschema")
-	(generator_version "8.0")
+	(generator_version "9.0")
 	(paper "User" 459.283 249.072)
+	(text "Base Address $E860"
+		(exclude_from_sim no)
+		(at 213.36 152.4 0)
+		(effects
+			(font
+				(size 1.9304 1.6408)
+			)
+			(justify left bottom)
+		)
+	)
+	(text "SID2 /CS for \nFPGASID with\nDual SIDs in SID1\nsocket"
+		(exclude_from_sim no)
+		(at 153.162 185.674 0)
+		(effects
+			(font
+				(size 1.27 1.27)
+			)
+		)
+	)
+	(text "CBM-ULTIPET-V1.1A\n"
+		(exclude_from_sim no)
+		(at 340.36 198.12 0)
+		(effects
+			(font
+				(size 3.81 3.2385)
+			)
+			(justify left bottom)
+		)
+	)
+	(text "SID 1\n"
+		(exclude_from_sim no)
+		(at 220.218 89.662 0)
+		(effects
+			(font
+				(size 1.27 1.27)
+			)
+		)
+	)
+	(text "CBM-ULTIPET-1.0A-20240331"
+		(exclude_from_sim no)
+		(at 337.82 220.98 0)
+		(effects
+			(font
+				(size 2.54 2.159)
+			)
+			(justify left bottom)
+		)
+	)
+	(text "Base Address $E8E0"
+		(exclude_from_sim no)
+		(at 213.36 218.44 0)
+		(effects
+			(font
+				(size 1.9304 1.6408)
+			)
+			(justify left bottom)
+		)
+	)
+	(text "SID 2"
+		(exclude_from_sim no)
+		(at 220.98 156.21 0)
+		(effects
+			(font
+				(size 1.27 1.27)
+			)
+		)
+	)
+	(text "C8,C11:\n22000pF for 8580\n470pF for 6581"
+		(exclude_from_sim no)
+		(at 231.14 86.36 0)
+		(effects
+			(font
+				(size 1.778 1.5113)
+			)
+			(justify left bottom)
+		)
+	)
+	(text "Absolutely only connect\nif only a single SID is\npopulated on the board!!!"
+		(exclude_from_sim no)
+		(at 287.782 130.81 0)
+		(effects
+			(font
+				(size 1.27 1.27)
+			)
+		)
+	)
+	(text "(C) A. Fachat"
+		(exclude_from_sim no)
+		(at 340.36 203.2 0)
+		(effects
+			(font
+				(size 2.54 2.159)
+			)
+			(justify left bottom)
+		)
+	)
+	(text "C15,C16:\n22000pF for 8580\n470pF for 6581"
+		(exclude_from_sim no)
+		(at 261.62 205.74 0)
+		(effects
+			(font
+				(size 1.778 1.5113)
+			)
+			(justify left bottom)
+		)
+	)
+	(text "8580 only, as only 9V\nare provided on VDD"
+		(exclude_from_sim no)
+		(at 363.22 182.88 0)
+		(effects
+			(font
+				(size 3.81 3.2385)
+			)
+			(justify left bottom)
+		)
+	)
+	(text "$E8Ex-$E8Fx"
+		(exclude_from_sim no)
+		(at 147.32 160.02 0)
+		(effects
+			(font
+				(size 1.778 1.5113)
+			)
+			(justify left bottom)
+		)
+	)
+	(text "Locate next to each other so\nDAC could be fed into extin"
+		(exclude_from_sim no)
+		(at 266.446 38.608 0)
+		(effects
+			(font
+				(size 1.27 1.27)
+			)
+		)
+	)
+	(text "$E86x-$E87x"
+		(exclude_from_sim no)
+		(at 147.32 157.48 0)
+		(effects
+			(font
+				(size 1.778 1.5113)
+			)
+			(justify left bottom)
+		)
+	)
 	(junction
 		(at 314.96 195.58)
@@
 		)
 	)
-	(text "Base Address $E860"
-		(exclude_from_sim no)
-		(at 213.36 152.4 0)
-		(effects
-			(font
-				(size 1.9304 1.6408)
-			)
-			(justify left bottom)
-		)
-	)
-	(text "SID2 /CS for \nFPGASID with\nDual SIDs in SID1\nsocket"
-		(exclude_from_sim no)
-		(at 153.162 185.674 0)
-		(effects
-			(font
-				(size 1.27 1.27)
-			)
-		)
-	)
-	(text "CBM-ULTIPET-V1.1A\n"
-		(exclude_from_sim no)
-		(at 340.36 198.12 0)
-		(effects
-			(font
-				(size 3.81 3.2385)
-			)
-			(justify left bottom)
-		)
-	)
-	(text "SID 1\n"
-		(exclude_from_sim no)
-		(at 220.218 89.662 0)
-		(effects
-			(font
-				(size 1.27 1.27)
-			)
-		)
-	)
-	(text "CBM-ULTIPET-1.0A-20240331"
-		(exclude_from_sim no)
-		(at 337.82 220.98 0)
-		(effects
-			(font
-				(size 2.54 2.159)
-			)
-			(justify left bottom)
-		)
-	)
-	(text "Base Address $E8E0"
-		(exclude_from_sim no)
-		(at 213.36 218.44 0)
-		(effects
-			(font
-				(size 1.9304 1.6408)
-			)
-			(justify left bottom)
-		)
-	)
-	(text "SID 2"
-		(exclude_from_sim no)
-		(at 220.98 156.21 0)
-		(effects
-			(font
-				(size 1.27 1.27)
-			)
-		)
-	)
-	(text "C8,C11:\n22000pF for 8580\n470pF for 6581"
-		(exclude_from_sim no)
-		(at 231.14 86.36 0)
-		(effects
-			(font
-				(size 1.778 1.5113)
-			)
-			(justify left bottom)
-		)
-	)
-	(text "Absolutely only connect\nif only a single SID is\npopulated on the board!!!"
-		(exclude_from_sim no)
-		(at 287.782 130.81 0)
-		(effects
-			(font
-				(size 1.27 1.27)
-			)
-		)
-	)
-	(text "(C) A. Fachat"
-		(exclude_from_sim no)
-		(at 340.36 203.2 0)
-		(effects
-			(font
-				(size 2.54 2.159)
-			)
-			(justify left bottom)
-		)
-	)
-	(text "C15,C16:\n22000pF for 8580\n470pF for 6581"
-		(exclude_from_sim no)
-		(at 261.62 205.74 0)
-		(effects
-			(font
-				(size 1.778 1.5113)
-			)
-			(justify left bottom)
-		)
-	)
-	(text "8580 only, as only 9V\nare provided on VDD"
-		(exclude_from_sim no)
-		(at 363.22 182.88 0)
-		(effects
-			(font
-				(size 3.81 3.2385)
-			)
-			(justify left bottom)
-		)
-	)
-	(text "$E8Ex-$E8Fx"
-		(exclude_from_sim no)
-		(at 147.32 160.02 0)
-		(effects
-			(font
-				(size 1.778 1.5113)
-			)
-			(justify left bottom)
-		)
-	)
-	(text "Locate next to each other so\nDAC could be fed into extin"
-		(exclude_from_sim no)
-		(at 266.446 38.608 0)
-		(effects
-			(font
-				(size 1.27 1.27)
-			)
-		)
-	)
-	(text "$E86x-$E87x"
-		(exclude_from_sim no)
-		(at 147.32 157.48 0)
-		(effects
-			(font
-				(size 1.778 1.5113)
-			)
-			(justify left bottom)
-		)
-	)
 	(global_label "V9V"
 		(shape input)
@@
 			)
 		)
-		(property "Footprint" "cbm_ultipet_v1:DIL16"
+		(property "Footprint" "Package_DIP:DIP-16_W7.62mm_Socket_LongPads"
 			(at 101.6 40.64 0)
 			(effects
@@
 			)
 		)
-		(property "Footprint" "cbm_ultipet_v1:DIL16"
+		(property "Footprint" "Package_DIP:DIP-16_W7.62mm_Socket_LongPads"
 			(at 154.94 146.05 0)
 			(effects
@@
 			)
 		)
-		(property "Footprint" "cbm_ultipet_v1:DIL16"
+		(property "Footprint" "Package_DIP:DIP-16_W7.62mm_Socket_LongPads"
 			(at 154.94 123.19 0)
 			(effects

Commit message: work on r1.3
Parts:
- U$22, U$23: footprint cbm_ultipet_v1:DIL28 -> Package_DIP:DIP-28_W15.24mm_Socket_LongPads
Changed lines of the file:
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@@
 			)
 		)
-		(property "Footprint" "cbm_ultipet_v1:DIL28"
+		(property "Footprint" "Package_DIP:DIP-28_W15.24mm_Socket_LongPads"
 			(at 223.52 180.34 0)
 			(effects
@@
 			)
 		)
-		(property "Footprint" "cbm_ultipet_v1:DIL28"
+		(property "Footprint" "Package_DIP:DIP-28_W15.24mm_Socket_LongPads"
 			(at 223.52 114.3 0)
 			(effects
