File: Board/UART.kicad_sch (KiCad schematic)
At the start: 23 parts, among them IC31 MAX232, IC32 MAX232, IC34 7406N, IC35 74138N, U8 74AHCT1G08, X3 M09HPS

Commit message: work on r1.3
Parts:
- removed U$2, U$27: JP5, cbm_ultipet_v1:JP5, symbol cbm_ultipet_v1-eagle-import:JP5
- added C157, C160: 100n, cbm_ultipet_v1:C0603, symbol cbm_ultipet_v1-eagle-import:C-EU025-024X044
- added J10, J11, J12: Conn_01x09, Connector_PinHeader_2.54mm:PinHeader_1x09_P2.54mm_Vertical, symbol Connector_Generic:Conn_01x09
- added J13: Conn_01x07, Connector_PinHeader_2.54mm:PinHeader_1x07_P2.54mm_Vertical, symbol Connector_Generic:Conn_01x07
- added R43, R44: 4k7, cbm_ultipet_v1:0207_10, symbol cbm_ultipet_v1-eagle-import:R-EU_0207/10
- added U10: CH340C, Package_SO:SOIC-16_3.9x9.9mm_P1.27mm, symbol Interface_USB:CH340C
Connections:
- net GND: now also C157.2, C160.2, J10.1 (Pin_1), J11.1 (Pin_1), J12.1 (Pin_1), J13.1 (Pin_1), R43.2, R44.2, U10.1 (GND); no longer IC6.29 (/DSRB), IC6.30 (/CDB)
- net LCTS: now also J12.2 (Pin_2)
- net LDCD: now also J12.8 (Pin_8)
- net LDSR: now also J12.6 (Pin_6)
- net LDTR: now also J12.7 (Pin_7)
- net LRTS: now also J12.5 (Pin_5)
- net LRX: now also J12.4 (Pin_4)
- net LTX: now also J12.3 (Pin_3)
- net RCTS: now also J11.2 (Pin_2)
- net RRTS: now also IC6.27 (/DTRB), J11.5 (Pin_5), J11.7 (Pin_7)
- net RRX: now also J11.4 (Pin_4)
- net RTX: now also J11.3 (Pin_3)
- net VCC: now also C160.1, U10.16 (VCC)
- net OPENHIGH renamed LRI
- net LRI: now also J12.9 (Pin_9); no longer IC6.31 (/RIB)
- new net: C157.1, U10.4 (V3)
- new net RCD: IC6.30 (/CDB), J11.8 (Pin_8), R43.1
- new net RDSR: IC6.29 (/DSRB), J11.6 (Pin_6), R44.1
- new net RRI: IC6.31 (/RIB), J11.9 (Pin_9)
- new net UCD: J10.8 (Pin_8), U10.12 (~{DCD})
- new net UCD+: U10.5 (UD+)
- new net UCD-: U10.6 (UD-)
- new net UCTS: J10.2 (Pin_2), J13.5 (Pin_5), U10.9 (~{CTS})
- new net UDSR: J10.6 (Pin_6), J13.7 (Pin_7), U10.10 (~{DSR})
- new net UDTR: J10.7 (Pin_7), J13.6 (Pin_6), U10.13 (~{DTR})
- new net URI: J10.9 (Pin_9), U10.11 (~{RI})
- new net URTS: J10.5 (Pin_5), J13.2 (Pin_2), U10.14 (~{RTS})
- new net URX: J10.4 (Pin_4), J13.3 (Pin_3), U10.3 (RXD)
- new net UTX: J10.3 (Pin_3), J13.4 (Pin_4), U10.2 (TXD)
Other:
- note added: "1.1A: - Switch to DUAL UART to provide 2nd 5V RS232 (shared w/ UEXT) - replace pullup on UART /RES with RN7 1.2A: - set /DSRB and /CDB to lo instead of hi . add pulldowns to INTA and INTB so high-Z does not trigger IRQ 1.3A: - Add USB-C RS232"
- note added: "CBM-ULTIPET-V1.3A"
- note added: "CBM-ULTIPET-V1.3A-20250806"
- note removed: "1.1A: - Switch to DUAL UART to provide 2nd 5V RS232 (shared w/ UEXT) - replace pullup on UART /RES with RN7 1.2A: - set /DSRB and /CDB to lo instead of hi . add pulldowns to INTA and INTB so high-Z does not trigger IRQ"
- note removed: "CBM-ULTIPET-V1.2A"
- note removed: "CBM-ULTIPET-V1.2A-20241013"
- moved on the sheet: C134, C135, C137, C139, C84, C86, C87, C88, C89, C90, C91, IC31A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
