File: Board/UART.kicad_sch (KiCad schematic)
At the start: 30 parts, among them IC31 MAX232, IC32 MAX232, IC34 7406N, IC35 74138N, J10 Conn_01x09, J11 Conn_01x09, J12 Conn_01x09, J13 Conn_01x07, U10 CH340C, U8 74AHCT1G08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

Commit message: more work on r1.3
Connections:
- net RRTS: no longer IC6.27 (/DTRB), J11.7 (Pin_7)
- new net RDTR: IC6.27 (/DTRB), J11.7 (Pin_7)
Changed lines of the file:
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@@
 		)
 	)
-	(label "RRTS"
+	(label "RDTR"
 		(at 246.38 172.72 90)
 		(effects

Commit message: preview for r1.3
Other:
- note added: "1.1A: - Switch to DUAL UART to provide 2nd 5V RS232 (shared w/ UEXT) - replace pullup on UART /RES with RN7 1.2A: - set /DSRB and /CDB to lo instead of hi . add pulldowns to INTA and INTB so high-Z does not trigger IRQ 1.3A: - Add USB-C RS232 - Extend internal connectors"
- note removed: "1.1A: - Switch to DUAL UART to provide 2nd 5V RS232 (shared w/ UEXT) - replace pullup on UART /RES with RN7 1.2A: - set /DSRB and /CDB to lo instead of hi . add pulldowns to INTA and INTB so high-Z does not trigger IRQ 1.3A: - Add USB-C RS232"
Changed lines of the file:
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@@
 		)
 	)
-	(text "1.1A:\n- Switch to DUAL UART to provide 2nd\n  5V RS232 (shared w/ UEXT)\n- replace pullup on UART /RES \n  with RN7\n1.2A:\n- set /DSRB and /CDB to lo instead of hi\n. add pulldowns to INTA and INTB so high-Z\n  does not trigger IRQ\n1.3A:\n- Add USB-C RS232"
+	(text "1.1A:\n- Switch to DUAL UART to provide 2nd\n  5V RS232 (shared w/ UEXT)\n- replace pullup on UART /RES \n  with RN7\n1.2A:\n- set /DSRB and /CDB to lo instead of hi\n. add pulldowns to INTA and INTB so high-Z\n  does not trigger IRQ\n1.3A:\n- Add USB-C RS232\n- Extend internal connectors"
 		(exclude_from_sim no)
 		(at 295.148 140.97 0)

Commit message: working on jlcpcb production files
Parts:
- IC6: value ~ -> 16255 UART
Changed lines of the file:
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@@
 			)
 		)
-		(property "Value" "~"
+		(property "Value" "16255 UART"
 			(at 173.9748 132.08 0)
 			(effects

Commit message: some layout fixes, more parts
Parts:
- C86, C87, C90, C91: footprint cbm_ultipet_v1:E2,5-6 -> cbm_ultipet_v1:E2-5
Changed lines of the file:
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@@
 			)
 		)
-		(property "Footprint" "cbm_ultipet_v1:E2,5-6"
+		(property "Footprint" "cbm_ultipet_v1:E2-5"
 			(at 198.12 30.48 0)
 			(effects
@@
 			)
 		)
-		(property "Footprint" "cbm_ultipet_v1:E2,5-6"
+		(property "Footprint" "cbm_ultipet_v1:E2-5"
 			(at 198.12 73.66 0)
 			(effects
@@
 			)
 		)
-		(property "Footprint" "cbm_ultipet_v1:E2,5-6"
+		(property "Footprint" "cbm_ultipet_v1:E2-5"
 			(at 198.12 40.64 0)
 			(effects
@@
 			)
 		)
-		(property "Footprint" "cbm_ultipet_v1:E2,5-6"
+		(property "Footprint" "cbm_ultipet_v1:E2-5"
 			(at 198.12 83.82 0)
 			(effects
