File: Board/Bus.kicad_sch (KiCad schematic)
At the start: 15 parts, among them IC13 74244DW, IC14 7414D, IC16 74LVC8T245SO24, IC18 7406D, IC19 74244DW, IC22 7400N, IC4 74245DW, IC5 74245DW, P1 CSABUSSOCK180

Commit message: ultipet 1.1a board
Parts:
- removed QG2: 16MHz, cbm_ultipet_v1:SG51, symbol cbm_ultipet_v1-eagle-import:CRYSTAL_RES-SG51
- removed R27: 10k, cbm_ultipet_v1:0204_5, symbol cbm_ultipet_v1-eagle-import:R-EU_0204/5
Connections:
- net C16M is gone; now on net OPENHIGH: IC19.4 (A2)
Other:
- note added: "1.0B: Removed the pullup on GRAPHIC, as it's now in the FPGA"
- note added: "CBM-ULTIPET-V1.1A"
- note added: "CSA-ULTIPET-V1.0B-20240502 (CSA-ULTRACPU-V1.3C-20231117)"
- note removed: "CBM-ULTIPET-V1.0A"
- note removed: "CSA-ULTRACPU-V1.3C-20231117"
- moved on the sheet: IC18G

Commit message: diverse fixes
Connections:
- net V33: no longer JP6.1
- new net V33IO: JP6.1
Other:
- note added: "1.0B: - Removed the pullup on GRAPHIC, as it's now in the FPGA 1.2A: - use V33IO for bus 3.3V (if so jumpered)"
- note added: "CBM-ULTIPET-V1.2A"
- note added: "CSA-ULTIPET-V1.2A-20241010"
- note removed: "1.0B: Removed the pullup on GRAPHIC, as it's now in the FPGA"
- note removed: "CBM-ULTIPET-V1.1A"
- note removed: "CSA-ULTIPET-V1.0B-20240502 (CSA-ULTRACPU-V1.3C-20231117)"
Changed lines of the file:
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@@
 	(wire
 		(pts
-			(xy 40.64 335.28) (xy 50.8 335.28)
-		)
-		(stroke
-			(width 0.1524)
-			(type solid)
-		)
-	)
-	(wire
-		(pts
 			(xy 86.36 304.8) (xy 104.14 304.8)
 		)
@@
 	(wire
 		(pts
+			(xy 40.64 332.74) (xy 40.64 322.58)
+		)
+		(stroke
+			(width 0)
+			(type default)
+		)
+	)
+	(wire
+		(pts
 			(xy 83.82 147.32) (xy 104.14 147.32)
 		)
@@
 	(wire
 		(pts
-			(xy 40.64 322.58) (xy 40.64 335.28)
-		)
-		(stroke
-			(width 0.1524)
-			(type solid)
-		)
-	)
-	(wire
-		(pts
 			(xy 40.64 294.64) (xy 40.64 297.18)
 		)
@@
 	(wire
 		(pts
+			(xy 41.91 332.74) (xy 40.64 332.74)
+		)
+		(stroke
+			(width 0)
+			(type default)
+		)
+	)
+	(wire
+		(pts
 			(xy 142.24 172.72) (xy 137.16 172.72)
 		)
@@
 		)
 	)
-	(text "CSA-ULTIPET-V1.0B-20240502\n(CSA-ULTRACPU-V1.3C-20231117)\n"
+	(text "CSA-ULTIPET-V1.2A-20241010\n"
 		(exclude_from_sim no)
-		(at 279.4 362.966 0)
+		(at 275.336 360.426 0)
 		(effects
 			(font
@@
 		)
 	)
-	(text "1.0B: Removed the pullup on GRAPHIC, as it's now in the FPGA"
+	(text "1.0B: \n- Removed the pullup on GRAPHIC, as it's now in the FPGA\n1.2A:\n- use V33IO for bus 3.3V (if so jumpered)"
 		(exclude_from_sim no)
-		(at 291.338 325.374 0)
+		(at 260.604 324.358 0)
 		(effects
 			(font
 				(size 1.7 1.7)
 			)
+			(justify left)
 		)
 	)
-	(text "CBM-ULTIPET-V1.1A"
+	(text "CBM-ULTIPET-V1.2A"
 		(exclude_from_sim no)
 		(at 254 337.82 0)
@@
 		)
 	)
+	(global_label "V33IO"
+		(shape input)
+		(at 41.91 332.74 0)
+		(fields_autoplaced yes)
+		(effects
+			(font
+				(size 1.27 1.27)
+			)
+			(justify left)
+		)
+		(property "Intersheetrefs" "${INTERSHEET_REFS}"
+			(at 50.3381 332.74 0)
+			(effects
+				(font
+					(size 1.27 1.27)
+				)
+				(justify left)
+				(hide yes)
+			)
+		)
+	)
 	(global_label "BA11"
 		(shape bidirectional)
@@
 			(effects
 				(font
-					(size 1.27 1.27)
-				)
-				(justify left)
-				(hide yes)
-			)
-		)
-	)
-	(global_label "V33"
-		(shape bidirectional)
-		(at 43.18 335.28 0)
-		(fields_autoplaced yes)
-		(effects
-			(font
-				(size 1.2446 1.2446)
-			)
-			(justify left)
-		)
-		(property "Intersheetrefs" "${INTERSHEET_REFS}"
-			(at 50.6316 335.28 0)
-			(effects
-				(font

Commit message: more fixes
Parts:
- IC14: value 7414D -> 74LVC14
- IC18: value 7406D -> 74LVC06
Changed lines of the file:
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@@
 			)
 		)
-		(property "Value" "7406D"
+		(property "Value" "74LVC06"
 			(at 215.9 78.74 0)
 			(effects
@@
 			)
 		)
-		(property "Value" "7414D"
+		(property "Value" "74LVC14"
 			(at 163.83 78.74 0)
 			(effects
@@
 			)
 		)
-		(property "Value" "7414D"
+		(property "Value" "74LVC14"
 			(at 163.83 48.26 0)
 			(effects
@@
 			)
 		)
-		(property "Value" "7414D"
+		(property "Value" "74LVC14"
 			(at 163.83 63.5 0)
 			(effects
@@
 			)
 		)
-		(property "Value" "7414D"
+		(property "Value" "74LVC14"
 			(at 163.83 93.98 0)
 			(effects
@@
 			)
 		)
-		(property "Value" "7414D"
+		(property "Value" "74LVC14"
 			(at 163.83 109.22 0)
 			(effects
@@
 			)
 		)
-		(property "Value" "7406D"
+		(property "Value" "74LVC06"
 			(at 215.9 109.22 0)
 			(effects
@@
 			)
 		)
-		(property "Value" "7406D"
+		(property "Value" "74LVC06"
 			(at 298.45 78.74 0)
 			(effects
@@
 			)
 		)
-		(property "Value" "7406D"
+		(property "Value" "74LVC06"
 			(at 160.02 114.3 0)
 			(effects
@@
 			)
 		)
-		(property "Value" "7406D"
+		(property "Value" "74LVC06"
 			(at 307.34 281.94 0)
 			(effects
@@
 			)
 		)
-		(property "Value" "7406D"
+		(property "Value" "74LVC06"
 			(at 210.82 114.3 0)
 			(effects
@@
 			)
 		)
-		(property "Value" "7406D"
+		(property "Value" "74LVC06"
 			(at 215.9 93.98 0)
 			(effects
@@
 			)
 		)
-		(property "Value" "7414D"
+		(property "Value" "74LVC14"
 			(at 308.61 78.74 0)
 			(effects
@@
 			)
 		)
-		(property "Value" "7414D"
+		(property "Value" "74LVC14"
 			(at 163.83 33.02 0)
 			(effects

Commit message: more layout work
Other:
- moved on the sheet: JP6
Changed lines of the file:
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@@
 	)
 	(junction
+		(at 50.8 317.5)
+		(diameter 0)
+		(color 0 0 0 0)
+	)
+	(junction
 		(at 307.34 81.28)
 		(diameter 0)
@@
 	(wire
 		(pts
-			(xy 43.18 327.66) (xy 50.8 327.66)
+			(xy 39.37 327.66) (xy 50.8 327.66)
 		)
 		(stroke
@@
 	(wire
 		(pts
-			(xy 43.18 322.58) (xy 43.18 327.66)
+			(xy 39.37 326.39) (xy 39.37 327.66)
 		)
 		(stroke
@@
 	(wire
 		(pts
-			(xy 40.64 332.74) (xy 40.64 322.58)
+			(xy 36.83 332.74) (xy 36.83 326.39)
 		)
 		(stroke
@@
 	(wire
 		(pts
-			(xy 41.91 332.74) (xy 40.64 332.74)
+			(xy 41.91 332.74) (xy 36.83 332.74)
 		)
 		(stroke
@@
 	(wire
 		(pts
+			(xy 40.64 317.5) (xy 50.8 317.5)
+		)
+		(stroke
+			(width 0.1524)
+			(type solid)
+		)
+	)
+	(wire
+		(pts
 			(xy 83.82 132.08) (xy 83.82 129.54)
 		)
@@
 		)
 	)
+	(global_label "BV33"
+		(shape output)
+		(at 40.64 317.5 180)
+		(fields_autoplaced yes)
+		(effects
+			(font
+				(size 1.27 1.27)
+			)
+			(justify right)
+		)
+		(property "Intersheetrefs" "${INTERSHEET_REFS}"
+			(at 32.8772 317.5 0)
+			(effects
+				(font
+					(size 1.27 1.27)
+				)
+				(justify right)
+				(hide yes)
+			)
+		)
+	)
 	(global_label "/BBE"
 		(shape bidirectional)
@@
 	(symbol
 		(lib_id "cbm_ultipet_v1-eagle-import:JP1E")
-		(at 40.64 320.04 0)
+		(at 36.83 323.85 0)
 		(unit 1)
 		(exclude_from_sim no)
@@
 		(dnp no)
 		(property "Reference" "JP6"
-			(at 39.37 320.04 90)
+			(at 35.56 323.85 90)
 			(effects
 				(font
@@
 		)
 		(property "Value" "JP1E"
-			(at 46.355 320.04 90)
+			(at 42.545 323.85 90)
 			(effects
 				(font
@@
 		)
 		(property "Footprint" "cbm_ultipet_v1:JP1"
-			(at 40.64 320.04 0)
+			(at 36.83 323.85 0)
 			(effects
 				(font
@@
 		)
 		(property "Datasheet" ""
-			(at 40.64 320.04 0)
+			(at 36.83 323.85 0)
 			(effects
 				(font
@@
 		)
 		(property "Description" ""
-			(at 40.64 320.04 0)
+			(at 36.83 323.85 0)
 			(effects
 				(font

Commit message: work on 1.3
Parts:
- IC13, IC19, IC4, IC5: footprint cbm_ultipet_v1:SO20W@1 -> Package_SO:SOP-20_7.5x12.8mm_P1.27mm
- IC22: footprint cbm_ultipet_v1:DIL14 -> Package_DIP:DIP-14_W7.62mm_Socket_LongPads
Changed lines of the file:
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@@
 (kicad_sch
-	(version 20231120)
+	(version 20250114)
 	(generator "eeschema")
-	(generator_version "8.0")
+	(generator_version "9.0")
 	(paper "User" 375.463 388.772)
+	(text "CSA-ULTIPET-V1.2A-20241010\n"
+		(exclude_from_sim no)
+		(at 275.336 360.426 0)
+		(effects
+			(font
+				(size 2 2)
+			)
+			(justify left bottom)
+		)
+	)
+	(text "5V side"
+		(exclude_from_sim no)
+		(at 38.1 109.22 0)
+		(effects
+			(font
+				(size 5.08 4.318)
+			)
+			(justify left bottom)
+		)
+	)
+	(text "(C) A. Fachat"
+		(exclude_from_sim no)
+		(at 254 342.9 0)
+		(effects
+			(font
+				(size 2.54 2.159)
+			)
+			(justify left bottom)
+		)
+	)
+	(text "3.3V side"
+		(exclude_from_sim no)
+		(at 276.86 109.22 0)
+		(effects
+			(font
+				(size 5.08 4.318)
+			)
+			(justify left bottom)
+		)
+	)
+	(text "1.0B: \n- Removed the pullup on GRAPHIC, as it's now in the FPGA\n1.2A:\n- use V33IO for bus 3.3V (if so jumpered)"
+		(exclude_from_sim no)
+		(at 260.604 324.358 0)
+		(effects
+			(font
+				(size 1.7 1.7)
+			)
+			(justify left)
+		)
+	)
+	(text "CBM-ULTIPET-V1.2A"
+		(exclude_from_sim no)
+		(at 254 337.82 0)
+		(effects
+			(font
+				(size 3.81 3.2385)
+			)
+			(justify left bottom)
+		)
+	)
 	(junction
 		(at 40.64 279.4)
@@
 		)
 	)
-	(text "CSA-ULTIPET-V1.2A-20241010\n"
-		(exclude_from_sim no)
-		(at 275.336 360.426 0)
-		(effects
-			(font
-				(size 2 2)
-			)
-			(justify left bottom)
-		)
-	)
-	(text "5V side"
-		(exclude_from_sim no)
-		(at 38.1 109.22 0)
-		(effects
-			(font
-				(size 5.08 4.318)
-			)
-			(justify left bottom)
-		)
-	)
-	(text "(C) A. Fachat"
-		(exclude_from_sim no)
-		(at 254 342.9 0)
-		(effects
-			(font
-				(size 2.54 2.159)
-			)
-			(justify left bottom)
-		)
-	)
-	(text "3.3V side"
-		(exclude_from_sim no)
-		(at 276.86 109.22 0)
-		(effects
-			(font
-				(size 5.08 4.318)
-			)
-			(justify left bottom)
-		)
-	)
-	(text "1.0B: \n- Removed the pullup on GRAPHIC, as it's now in the FPGA\n1.2A:\n- use V33IO for bus 3.3V (if so jumpered)"
-		(exclude_from_sim no)
-		(at 260.604 324.358 0)
-		(effects
-			(font
-				(size 1.7 1.7)
-			)
-			(justify left)
-		)
-	)
-	(text "CBM-ULTIPET-V1.2A"
-		(exclude_from_sim no)
-		(at 254 337.82 0)
-		(effects
-			(font
-				(size 3.81 3.2385)
-			)
-			(justify left bottom)
-		)
-	)
 	(label "/BEXTIO"
 		(at 106.68 121.92 90)
@@
 			)
 		)
-		(property "Footprint" "cbm_ultipet_v1:SO20W@1"
+		(property "Footprint" "Package_SO:SOP-20_7.5x12.8mm_P1.27mm"
 			(at 259.08 294.64 0)
 			(effects
@@
 			)
 		)
-		(property "Footprint" "cbm_ultipet_v1:SO20W@1"
+		(property "Footprint" "Package_SO:SOP-20_7.5x12.8mm_P1.27mm"
 			(at 160.02 297.18 0)
 			(effects
@@
 			)
 		)
-		(property "Footprint" "cbm_ultipet_v1:SO20W@1"
+		(property "Footprint" "Package_SO:SOP-20_7.5x12.8mm_P1.27mm"
 			(at 160.02 332.74 0)
 			(effects
@@
 			)
 		)
-		(property "Footprint" "cbm_ultipet_v1:DIL14"
+		(property "Footprint" "Package_DIP:DIP-14_W7.62mm_Socket_LongPads"
 			(at 55.88 185.42 0)
 			(effects
@@
 			)
 		)
-		(property "Footprint" "cbm_ultipet_v1:SO20W@1"
+		(property "Footprint" "Package_SO:SOP-20_7.5x12.8mm_P1.27mm"
 			(at 160.02 238.76 0)
 			(effects
@@
 			)
 		)
-		(property "Footprint" "cbm_ultipet_v1:SO20W@1"
+		(property "Footprint" "Package_SO:SOP-20_7.5x12.8mm_P1.27mm"
 			(at 307.34 243.84 0)
 			(effects
@@
 			)
 		)
-		(property "Footprint" "cbm_ultipet_v1:SO20W@1"
+		(property "Footprint" "Package_SO:SOP-20_7.5x12.8mm_P1.27mm"
 			(at 160.02 200.66 0)
 			(effects
@@
 			)
 		)
-		(property "Footprint" "cbm_ultipet_v1:SO20W@1"
+		(property "Footprint" "Package_SO:SOP-20_7.5x12.8mm_P1.27mm"
 			(at 228.6 294.64 0)
 			(effects
@@
 			)
 		)
-		(property "Footprint" "cbm_ultipet_v1:SO20W@1"
+		(property "Footprint" "Package_SO:SOP-20_7.5x12.8mm_P1.27mm"
 			(at 248.92 294.64 0)
 			(effects
@@
 			)
 		)
-		(property "Footprint" "cbm_ultipet_v1:SO20W@1"
+		(property "Footprint" "Package_SO:SOP-20_7.5x12.8mm_P1.27mm"
 			(at 160.02 266.7 0)
 			(effects
@@
 			)
 		)
-		(property "Footprint" "cbm_ultipet_v1:SO20W@1"
+		(property "Footprint" "Package_SO:SOP-20_7.5x12.8mm_P1.27mm"
 			(at 238.76 294.64 0)
 			(effects

Commit message: preview for r1.3
Other:
- note added: "CBM-ULTIPET-V1.3A"
- note removed: "CBM-ULTIPET-V1.2A"
Changed lines of the file:
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@@
 		)
 	)
-	(text "CBM-ULTIPET-V1.2A"
+	(text "CBM-ULTIPET-V1.3A"
 		(exclude_from_sim no)
 		(at 254 337.82 0)
