File: Board/Userport.kicad_sch (KiCad schematic)
At the start: 31 parts, among them CN5 PORT_USER_PET_EDGE, U4 CD4053B, U5 CD4053B, X7 M09-182, X8 M09-182

Commit message: preview for r1.3
Other:
- note added: "1.1A: - switch between single/dual joystick config - switch Joy1/Joy2 on board 1.2A: - switch diodes direction to fix dual mode joystick fire - replace 1N4148 with 1N4448 due to lower fwd voltage - add clamping diodes to joystick port 1.3A: - fix joystick connector footprint"
- note added: "CBM-ULTIPET-V1.3A"
- note added: "CBM-ULTIPET-V1.3A-20250806"
- note removed: "1.1A: - switch between single/dual joystick config - switch Joy1/Joy2 on board 1.2A: - switch diodes direction to fix dual mode joystick fire - replace 1N4148 with 1N4448 due to lower fwd voltage - add clamping diodes to joystick port"
- note removed: "CBM-ULTIPET-V1.2A"
- note removed: "CBM-ULTIPET-V1.2A-20241017"
Changed lines of the file:
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@@
 		)
 	)
-	(text "1.1A:\n- switch between single/dual joystick config\n- switch Joy1/Joy2 on board\n1.2A:\n- switch diodes direction to fix dual mode joystick fire\n- replace 1N4148 with 1N4448 due to lower fwd voltage\n- add clamping diodes to joystick port"
+	(text "1.1A:\n- switch between single/dual joystick config\n- switch Joy1/Joy2 on board\n1.2A:\n- switch diodes direction to fix dual mode joystick fire\n- replace 1N4148 with 1N4448 due to lower fwd voltage\n- add clamping diodes to joystick port\n1.3A:\n- fix joystick connector footprint"
 		(exclude_from_sim no)
 		(at 189.484 35.56 0)
@@
 		)
 	)
-	(text "CBM-ULTIPET-V1.2A"
+	(text "CBM-ULTIPET-V1.3A"
 		(exclude_from_sim no)
 		(at 187.96 160.02 0)
@@
 		)
 	)
-	(text "CBM-ULTIPET-V1.2A-20241017"
+	(text "CBM-ULTIPET-V1.3A-20250806"
 		(exclude_from_sim no)
 		(at 190.5 180.34 0)
