File: Board/A%2fV.kicad_sch (KiCad schematic)
At the start: 24 parts, among them IC2 74245DW, X2 D-SUB15-HDR15RA

Commit message: preview for r1.3
Other:
- note added: "1.2A: - add Digital Video Out connector 1.3A: - VGA footprint with solderable supports"
- note added: "CBM-ULTIPET-V1.3A"
- note added: "CSA-ULTIPET-V1.3A-20250806"
- note removed: "1.2A: - add Digital Video Out connector"
- note removed: "CBM-ULTIPET-V1.2A"
- note removed: "CSA-ULTIPET-V1.2A-20241115"
Changed lines of the file:
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@@
 	(generator_version "9.0")
 	(paper "User" 334.823 210.007)
-	(text "1.2A:\n- add Digital Video Out connector"
+	(text "1.2A:\n- add Digital Video Out connector\n1.3A:\n- VGA footprint with solderable supports"
 		(exclude_from_sim no)
-		(at 224.282 132.588 0)
+		(at 222.25 127 0)
 		(effects
 			(font
@@
 		)
 	)
-	(text "CSA-ULTIPET-V1.2A-20241115"
+	(text "CSA-ULTIPET-V1.3A-20250806"
 		(exclude_from_sim no)
 		(at 208.28 167.64 0)
@@
 		)
 	)
-	(text "CBM-ULTIPET-V1.2A"
+	(text "CBM-ULTIPET-V1.3A"
 		(exclude_from_sim no)
 		(at 208.28 144.78 0)

Commit message: new USB C conn; BOM work
Parts:
- C73, C94: footprint cbm_ultipet_v1:C025-024X044 -> cbm_ultipet_v1:C025-025X050
Changed lines of the file:
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@@
 			)
 		)
-		(property "Footprint" "cbm_ultipet_v1:C025-024X044"
+		(property "Footprint" "cbm_ultipet_v1:C025-025X050"
 			(at 279.4 68.58 0)
 			(effects
@@
 			)
 		)
-		(property "Footprint" "cbm_ultipet_v1:C025-024X044"
+		(property "Footprint" "cbm_ultipet_v1:C025-025X050"
 			(at 287.02 68.58 0)
 			(effects

Commit message: rename U refs to UX*
Parts:
- renumbered U$10 to UX10, U$11 to UX11, U$5 to UX5, U$6 to UX6, U$8 to UX8
Changed lines of the file:
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@@
 		(on_board yes)
 		(dnp no)
-		(property "Reference" "U$5"
+		(property "Reference" "UX5"
 			(at 189.865 153.162 0)
 			(effects
@@
 			(project "cbm_ultipet_v1"
 				(path "/4dd2dd78-173f-4b46-8cce-4ed940435c94/122e60a4-4a83-4478-ae42-3d8b51948846"
-					(reference "U$5")
+					(reference "UX5")
 					(unit 1)
 				)
@@
 		(on_board yes)
 		(dnp no)
-		(property "Reference" "U$8"
+		(property "Reference" "UX8"
 			(at 174.625 153.162 0)
 			(effects
@@
 			(project "cbm_ultipet_v1"
 				(path "/4dd2dd78-173f-4b46-8cce-4ed940435c94/122e60a4-4a83-4478-ae42-3d8b51948846"
-					(reference "U$8")
+					(reference "UX8")
 					(unit 1)
 				)
@@
 		(on_board yes)
 		(dnp no)
-		(property "Reference" "U$6"
+		(property "Reference" "UX6"
 			(at 182.245 153.162 0)
 			(effects
@@
 			(project "cbm_ultipet_v1"
 				(path "/4dd2dd78-173f-4b46-8cce-4ed940435c94/122e60a4-4a83-4478-ae42-3d8b51948846"
-					(reference "U$6")
+					(reference "UX6")
 					(unit 1)
 				)
@@
 		(on_board yes)
 		(dnp no)
-		(property "Reference" "U$11"
+		(property "Reference" "UX11"
 			(at 159.385 153.162 0)
 			(effects
@@
 			(project "cbm_ultipet_v1"
 				(path "/4dd2dd78-173f-4b46-8cce-4ed940435c94/122e60a4-4a83-4478-ae42-3d8b51948846"
-					(reference "U$11")
+					(reference "UX11")
 					(unit 1)
 				)
@@
 		(on_board yes)
 		(dnp no)
-		(property "Reference" "U$10"
+		(property "Reference" "UX10"
 			(at 167.005 153.162 0)
 			(effects
@@
 			(project "cbm_ultipet_v1"
 				(path "/4dd2dd78-173f-4b46-8cce-4ed940435c94/122e60a4-4a83-4478-ae42-3d8b51948846"
-					(reference "U$10")
+					(reference "UX10")
 					(unit 1)
 				)
