File: Board/FastIEC.kicad_sch (KiCad schematic)
At the start: 19 parts, among them IC21 7417N, IC23 7486N, IC34 7406N, IC36 VIA, IC40 7474N, IC48 7414N, IC49 74241N

Commit message: ultipet 1.1a board
Parts:
- removed unit 5 of IC34
- removed unit 4 of IC48
- removed JP30: JP6Q, cbm_ultipet_v1:JP6Q, symbol cbm_ultipet_v1-eagle-import:JP6Q
- added C145: 100n, cbm_ultipet_v1:C025-024X044, symbol cbm_ultipet_v1-eagle-import:C-EU025-024X044
- added unit 2 of IC21
- added J8: Conn_02x04_Odd_Even, Connector_PinHeader_2.54mm:PinHeader_2x04_P2.54mm_Vertical, symbol Connector_Generic:Conn_02x04_Odd_Even
- added P9: ~, Connector_IDC:IDC-Header_2x05_P2.54mm_Vertical, symbol SPI:SPI-10-5V
- added U2: 74HCT164, Package_DIP:DIP-14_W7.62mm_LongPads, symbol 74xx:74HCT164
- added U3: 74HCT00, cbm_ultipet_v1:DIL14, symbol 74xx:74HCT00
Connections:
- net CLKOUT: now also P9.4 (AUX)
- net DATA: now also IC21.2 (O)
- net DATAOUT: now also IC48.3 (I)
- net DFASTIECCLK: now also IC48.5 (I), J8.1 (Pin_1), U2.8 (CP), U3.10, U3.5
- net FASTIECDATA: now also P9.8 (MOSI)
- net FUC1: now also P9.6 (/IRQ)
- net FUC2: now also U3.1
- net FUP0: now also U2.3 (Q0)
- net FUP1: now also U2.4 (Q1)
- net FUP2: now also U2.5 (Q2)
- net FUP3: now also U2.6 (Q3)
- net FUP4: now also U2.10 (Q4)
- net FUP5: now also U2.11 (Q5)
- net FUP6: now also U2.12 (Q6)
- net FUP7: now also U2.13 (Q7)
- net GND: now also C145.2, P9.2 (GND), U2.7 (GND), U3.7 (GND)
- net OPENHIGH: no longer IC48.3 (I), IC48.5 (I)
- net VCC: now also C145.1, P9.1 (VCC), U2.1 (DSA), U2.14 (VCC), U2.9 (~{MR}), U3.14 (VCC)
- net at IC48.4 (O): now also IC21.1 (I), P9.10 (/SEL)
- net at IC48.6 (O): now also J8.5 (Pin_5)
- new net: U3.3, U3.4
- new net: U3.2, U3.6, U3.9
- new net: P9.7 (MISO), U2.2 (DSB)
- new net: J8.7 (Pin_7), U3.11
- new net: J8.3 (Pin_3), U3.12, U3.13, U3.8
- new net: J8.2 (Pin_2), J8.4 (Pin_4), J8.6 (Pin_6), J8.8 (Pin_8), P9.9 (CLK)
- new net /BRES: P9.5 (/RES)
Other:
- note added: "1.1A: - Add VIA/HW SR SPI for SPI-10-5V connector - Replace discrete R with RN7 on PULLUP_FUC1"
- note added: "CBM-ULTIPET-V1.1A"
- note added: "CBM-ULTIPET-V1.1A-20240614"
- note added: "Mode select jumper (3-0)"
- note added: "Test points / Internal drive"
- note added: "To pullup"
- note added: "http://forum.6502.org/viewtopic.php?f=4&t=7937#p106623"
- note removed: "CBM-ULTIPET-V1.0A"
- note removed: "CBM-ULTIPET-V1.0A-20240104"
- note removed: "Free Userports for experiments"
- note removed: "Note: IC49A is required, as VIA SR data out stays at last bit level."
- moved on the sheet: D14, IC36A, IC48E, IC48F

Commit message: various fixes as documented in github issues
Parts:
- removed JP31: JP2E, cbm_ultipet_v1:JP2, symbol cbm_ultipet_v1-eagle-import:JP2E
- added JP5: SolderJumper_3_Bridged12, Jumper:SolderJumper-3_P1.3mm_Bridged12_RoundedPad1.0x1.5mm_NumberLabels, symbol Jumper:SolderJumper_3_Bridged12
- D14: value 1N4148DO35-7 -> 1N4448
Connections:
- net DFASTIECCLK: now also JP5.2 (C)
- net FASTIECCLK: now also JP5.3 (B)
- net at IC49.7 (Y2): now also JP5.1 (A)
Other:
- note added: "1.1A: - Add VIA/HW SR SPI for SPI-10-5V connector - Replace discrete R with RN7 on PULLUP_FUC1 1.2A: - replace pin jumper for VIA fix with solder jumper - replace 1N4148 with 1N4448 for lower fwd voltage"
- note added: "CBM-ULTIPET-V1.2A"
- note added: "CBM-ULTIPET-V1.2A-20241013"
- note removed: "1.1A: - Add VIA/HW SR SPI for SPI-10-5V connector - Replace discrete R with RN7 on PULLUP_FUC1"
- note removed: "CBM-ULTIPET-V1.1A"
- note removed: "CBM-ULTIPET-V1.1A-20240614"
Changed lines of the file:
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@@
 	(wire
 		(pts
+			(xy 241.3 170.18) (xy 241.3 166.37)
+		)
+		(stroke
+			(width 0.1524)
+			(type solid)
+		)
+	)
+	(wire
+		(pts
 			(xy 143.51 120.65) (xy 143.51 160.02)
 		)
@@
 	(wire
 		(pts
-			(xy 256.54 165.1) (xy 256.54 170.18)
-		)
-		(stroke
-			(width 0.1524)
-			(type solid)
-		)
-	)
-	(wire
-		(pts
 			(xy 134.62 58.42) (xy 142.24 58.42)
 		)
@@
 	(wire
 		(pts
-			(xy 259.08 165.1) (xy 259.08 167.64)
-		)
-		(stroke
-			(width 0.1524)
-			(type solid)
-		)
-	)
-	(wire
-		(pts
 			(xy 309.88 96.52) (xy 317.5 96.52)
 		)
@@
 	(wire
 		(pts
+			(xy 246.38 167.64) (xy 246.38 162.56)
+		)
+		(stroke
+			(width 0.1524)
+			(type solid)
+		)
+	)
+	(wire
+		(pts
 			(xy 312.42 124.46) (xy 322.58 124.46)
 		)
@@
 	(wire
 		(pts
+			(xy 236.22 172.72) (xy 236.22 162.56)
+		)
+		(stroke
+			(width 0.1524)
+			(type solid)
+		)
+	)
+	(wire
+		(pts
 			(xy 205.74 156.21) (xy 214.63 156.21)
 		)
@@
 	(wire
 		(pts
-			(xy 256.54 170.18) (xy 269.24 170.18)
+			(xy 241.3 170.18) (xy 269.24 170.18)
 		)
 		(stroke
@@
 	(wire
 		(pts
-			(xy 254 172.72) (xy 254 165.1)
-		)
-		(stroke
-			(width 0.1524)
-			(type solid)
-		)
-	)
-	(wire
-		(pts
 			(xy 317.5 96.52) (xy 317.5 74.93)
 		)
@@
 	(wire
 		(pts
-			(xy 266.7 172.72) (xy 254 172.72)
+			(xy 236.22 172.72) (xy 266.7 172.72)
 		)
 		(stroke
@@
 	(wire
 		(pts
+			(xy 246.38 167.64) (xy 271.78 167.64)
+		)
+		(stroke
+			(width 0.1524)
+			(type solid)
+		)
+	)
+	(wire
+		(pts
 			(xy 73.66 33.02) (xy 83.82 33.02)
 		)
@@
 	(wire
 		(pts
-			(xy 259.08 167.64) (xy 271.78 167.64)
-		)
-		(stroke
-			(width 0.1524)
-			(type solid)
-		)
-	)
-	(wire
-		(pts
 			(xy 134.62 48.26) (xy 134.62 58.42)
 		)
@@
 		)
 	)
-	(text "CBM-ULTIPET-V1.1A\n"
+	(text "CBM-ULTIPET-V1.2A\n"
 		(exclude_from_sim no)
 		(at 27.94 195.58 0)
@@
 		)
 	)
-	(text "CBM-ULTIPET-V1.1A-20240614"
+	(text "CBM-ULTIPET-V1.2A-20241013"
 		(exclude_from_sim no)
 		(at 30.48 215.9 0)
@@
 		)
 	)
-	(text "1.1A:\n- Add VIA/HW SR SPI for SPI-10-5V connector\n- Replace discrete R with RN7 on PULLUP_FUC1"
+	(text "1.1A:\n- Add VIA/HW SR SPI for SPI-10-5V connector\n- Replace discrete R with RN7 on PULLUP_FUC1\n1.2A:\n- replace pin jumper for VIA fix with solder jumper\n- replace 1N4148 with 1N4448 for lower fwd voltage"
 		(exclude_from_sim no)
-		(at 131.064 212.344 0)
+		(at 131.572 209.042 0)
 		(effects
 			(font
@@
 	)
 	(symbol
-		(lib_id "cbm_ultipet_v1-eagle-import:JP2E")
-		(at 256.54 162.56 0)
-		(unit 1)
-		(exclude_from_sim no)
-		(in_bom yes)
-		(on_board yes)
-		(dnp no)
-		(property "Reference" "JP31"
-			(at 252.73 162.56 90)
-			(effects
-				(font
-					(size 1.778 1.5113)
-				)
-				(justify left bottom)
-			)
-		)
-		(property "Value" "JP2E"
-			(at 262.255 162.56 90)
-			(effects
-				(font
-					(size 1.778 1.5113)
-				)
-				(justify left bottom)
-				(hide yes)
-			)
-		)
-		(property "Footprint" "cbm_ultipet_v1:JP2"
-			(at 256.54 162.56 0)
-			(effects
-				(font
-					(size 1.27 1.27)
-				)
-				(hide yes)
-			)
-		)
-		(property "Datasheet" ""
-			(at 256.54 162.56 0)
-			(effects
-				(font
-					(size 1.27 1.27)
-				)
-				(hide yes)
-			)
-		)
-		(property "Description" ""
-			(at 256.54 162.56 0)
-			(effects
-				(font
-					(size 1.27 1.27)
-				)
-				(hide yes)
-			)
-		)
-		(pin "2"
-		)
-		(pin "1"
-		)
-		(pin "3"
-		)
-		(instances
-			(project "cbm_ultipet_v1"
-				(path "/4dd2dd78-173f-4b46-8cce-4ed940435c94/d6afba7b-0912-4ee1-adba-d44a9d4919d9"
-					(reference "JP31")
-					(unit 1)
-				)
-			)
-		)
-	)
-	(symbol
 		(lib_id "cbm_ultipet_v1-eagle-import:7417N")
 		(at 241.3 90.17 0)
@@
 			)
 		)
-		(property "Value" "1N4148DO35-7"
+		(property "Value" "1N4448"
 			(at 34.29 98.8314 0)
 			(effects
@@
 				)
 			)
+		)
+	)
+	(symbol
+		(lib_id "Jumper:SolderJumper_3_Bridged12")
+		(at 241.3 162.56 0)
+		(unit 1)
+		(exclude_from_sim yes)
+		(in_bom no)
+		(on_board yes)
+		(dnp no)
+		(property "Reference" "JP5"
+			(at 241.3 160.274 0)
+			(effects
+				(font
+					(size 1.27 1.27)
+				)
+			)
+		)
+		(property "Value" "SolderJumper_3_Bridged12"
+			(at 245.364 157.48 0)
+			(effects
+				(font
+					(size 1.27 1.27)
+				)
+			)
+		)
+		(property "Footprint" "Jumper:SolderJumper-3_P1.3mm_Bridged12_RoundedPad1.0x1.5mm_NumberLabels"
+			(at 241.3 162.56 0)
+			(effects
+				(font
+					(size 1.27 1.27)
+				)
+				(hide yes)
+			)
+		)
+		(property "Datasheet" "~"
+			(at 241.3 162.56 0)
+			(effects
+				(font
+					(size 1.27 1.27)
+				)
+				(hide yes)
+			)
+		)
+		(property "Description" "3-pole Solder Jumper, pins 1+2 closed/bridged"
+			(at 241.3 162.56 0)
+			(effects
+				(font
+					(size 1.27 1.27)
+				)
+				(hide yes)
+			)
+		)
+		(pin "1"
+		)
+		(pin "3"
+		)
+		(pin "2"
+		)
+		(instances
+			(project "cbm_ultipet_v1"
+				(path "/4dd2dd78-173f-4b46-8cce-4ed940435c94/d6afba7b-0912-4ee1-adba-d44a9d4919d9"
+					(reference "JP5")
+					(unit 1)
+				)
+			)

Commit message: work on 1.3
Parts:
- IC21, IC23, IC34, IC40, IC48, U3: footprint cbm_ultipet_v1:DIL14 -> Package_DIP:DIP-14_W7.62mm_Socket_LongPads
- IC36: footprint cbm_ultipet_v1:DIL40 -> Package_DIP:DIP-42_W15.24mm_Socket_LongPads
- IC49: footprint cbm_ultipet_v1:DIL20 -> Package_DIP:DIP-20_W7.62mm_Socket_LongPads
- U2: footprint Package_DIP:DIP-14_W7.62mm_LongPads -> Package_DIP:DIP-14_W7.62mm_Socket_LongPads

Commit message: preview for r1.3
Other:
- note added: "CBM-ULTIPET-V1.3A"
- note removed: "CBM-ULTIPET-V1.2A"
Changed lines of the file:
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@@
 		)
 	)
-	(text "CBM-ULTIPET-V1.2A\n"
+	(text "CBM-ULTIPET-V1.3A\n"
 		(exclude_from_sim no)
 		(at 27.94 195.58 0)

Commit message: more layout work on r1.3
Parts:
- IC36: footprint Package_DIP:DIP-42_W15.24mm_Socket_LongPads -> Package_DIP:DIP-40_W15.24mm_Socket_LongPads
Changed lines of the file:
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@@
 			)
 		)
-		(property "Footprint" "Package_DIP:DIP-42_W15.24mm_Socket_LongPads"
+		(property "Footprint" "Package_DIP:DIP-40_W15.24mm_Socket_LongPads"
 			(at 111.76 58.42 0)
 			(effects
@@
 			)
 		)
-		(property "Footprint" "Package_DIP:DIP-42_W15.24mm_Socket_LongPads"
+		(property "Footprint" "Package_DIP:DIP-40_W15.24mm_Socket_LongPads"
 			(at 80.01 132.08 0)
 			(effects

Commit message: rename U refs to UX*
Parts:
- renumbered U$28 to UX28
Changed lines of the file:
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@@
 		(on_board yes)
 		(dnp no)
-		(property "Reference" "U$28"
+		(property "Reference" "UX28"
 			(at 284.48 80.645 0)
 			(effects
@@
 			(project "cbm_ultipet_v1"
 				(path "/4dd2dd78-173f-4b46-8cce-4ed940435c94/d6afba7b-0912-4ee1-adba-d44a9d4919d9"
-					(reference "U$28")
+					(reference "UX28")
 					(unit 1)
 				)
