File: Board/Keylock.kicad_sch (KiCad schematic)
At the start: 20 parts, among them IC27 7474N, IC28 74138N, IC29 556N, Q1 BC557, T10 BC547

Commit message: ultipet 1.1a board
Other:
- note added: "CBM-ULTIPET-V1.1A"
- note removed: "CBM-ULTIPET1.0A"
Changed lines of the file:
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@@
 		)
 	)
-	(text "CBM-ULTIPET1.0A"
+	(text "CBM-ULTIPET-V1.1A"
 		(exclude_from_sim no)
 		(at 25.4 160.02 0)

Commit message: diverse fixes
Connections:
- net KEYLOCK: now reaches IC27.12 (D), IC27.8 (~{Q})
Other:
- note added: "CBM-ULTIPET-1.2A-20241010"
- note added: "CBM-ULTIPET-V1.2A"
- note added: "R1.2A: - add KEYLOCK_LED output"
- note removed: "CBM-KEYLOCK-1.0B-20240104"
- note removed: "CBM-ULTIPET-V1.1A"
Changed lines of the file:
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@@
+	)
+	(junction
+		(at 208.28 54.61)
+		(diameter 0)
+		(color 0 0 0 0)
 	)
 	(junction
@@
 	(wire
 		(pts
+			(xy 208.28 54.61) (xy 222.25 54.61)
+		)
+		(stroke
+			(width 0.1524)
+			(type solid)
+		)
+	)
+	(wire
+		(pts
 			(xy 167.64 162.56) (xy 177.8 162.56)
 		)
@@
 	(wire
 		(pts
+			(xy 208.28 54.61) (xy 208.28 53.34)
+		)
+		(stroke
+			(width 0.1524)
+			(type solid)
+		)
+	)
+	(wire
+		(pts
 			(xy 256.54 83.82) (xy 264.16 83.82)
 		)
@@
 	(wire
 		(pts
-			(xy 208.28 73.66) (xy 208.28 53.34)
+			(xy 208.28 73.66) (xy 208.28 54.61)
 		)
 		(stroke
@@
 		)
 	)
-	(text "CBM-ULTIPET-V1.1A"
+	(text "CBM-ULTIPET-V1.2A"
 		(exclude_from_sim no)
 		(at 25.4 160.02 0)
@@
 		)
 	)
-	(text "CBM-KEYLOCK-1.0B-20240104"
+	(text "CBM-ULTIPET-1.2A-20241010"
 		(exclude_from_sim no)
 		(at 25.4 177.8 0)
@@
 			)
 			(justify left bottom)
+		)
+	)
+	(text "R1.2A:\n- add KEYLOCK_LED output"
+		(exclude_from_sim no)
+		(at 233.172 172.72 0)
+		(effects
+			(font
+				(size 2.54 2.54)
+			)
+			(justify left)
 		)
 	)
@@
 			(effects
 				(font
+					(size 1.27 1.27)
+				)
+				(justify left)
+				(hide yes)
+			)
+		)
+	)
+	(global_label "KEYLOCK"
+		(shape output)
+		(at 222.25 54.61 0)
+		(fields_autoplaced yes)
+		(effects
+			(font
+				(size 1.27 1.27)
+			)
+			(justify left)
+		)
+		(property "Intersheetrefs" "${INTERSHEET_REFS}"
+			(at 233.6414 54.61 0)
+			(effects
+				(font

Commit message: work on 1.3
Parts:
- IC27, IC29: footprint cbm_ultipet_v1:DIL14 -> Package_DIP:DIP-14_W7.62mm_Socket_LongPads
- IC28: footprint cbm_ultipet_v1:DIL16 -> Package_DIP:DIP-16_W7.62mm_Socket_LongPads
Changed lines of the file:
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@@
 (kicad_sch
-	(version 20231120)
+	(version 20250114)
 	(generator "eeschema")
-	(generator_version "8.0")
+	(generator_version "9.0")
 	(paper "User" 317.652 210.007)
+	(text "Commodore PET SHIFT-LOCK simulator + RESET on long push"
+		(exclude_from_sim no)
+		(at 22.86 33.02 0)
+		(effects
+			(font
+				(size 3.81 3.2385)
+			)
+			(justify left bottom)
+		)
+	)
+	(text "CBM-ULTIPET-V1.2A"
+		(exclude_from_sim no)
+		(at 25.4 160.02 0)
+		(effects
+			(font
+				(size 3.81 3.2385)
+			)
+			(justify left bottom)
+		)
+	)
+	(text "Business"
+		(exclude_from_sim no)
+		(at 78.74 99.06 90)
+		(effects
+			(font
+				(size 1.778 1.5113)
+			)
+			(justify left bottom)
+		)
+	)
+	(text "Business"
+		(exclude_from_sim no)
+		(at 129.54 111.76 90)
+		(effects
+			(font
+				(size 1.778 1.5113)
+			)
+			(justify left bottom)
+		)
+	)
+	(text "Business"
+		(exclude_from_sim no)
+		(at 165.1 111.76 90)
+		(effects
+			(font
+				(size 1.778 1.5113)
+			)
+			(justify left bottom)
+		)
+	)
+	(text "Low = no key,\nhigh = key pressed"
+		(exclude_from_sim no)
+		(at 142.24 134.62 0)
+		(effects
+			(font
+				(size 1.778 1.5113)
+			)
+			(justify left bottom)
+		)
+	)
+	(text "Business"
+		(exclude_from_sim no)
+		(at 287.02 104.14 90)
+		(effects
+			(font
+				(size 1.778 1.5113)
+			)
+			(justify left bottom)
+		)
+	)
+	(text "Graphics"
+		(exclude_from_sim no)
+		(at 271.78 104.14 90)
+		(effects
+			(font
+				(size 1.778 1.5113)
+			)
+			(justify left bottom)
+		)
+	)
+	(text "/RES is 3.3V from CPU\nside. That then triggers\n/BRES on 5V side"
+		(exclude_from_sim no)
+		(at 195.58 137.16 0)
+		(effects
+			(font
+				(size 1.778 1.5113)
+			)
+			(justify left bottom)
+		)
+	)
+	(text "CBM-ULTIPET-1.2A-20241010"
+		(exclude_from_sim no)
+		(at 25.4 177.8 0)
+		(effects
+			(font
+				(size 2.54 2.159)
+			)
+			(justify left bottom)
+		)
+	)
+	(text "Saves the last\nkey press state"
+		(exclude_from_sim no)
+		(at 101.6 55.88 0)
+		(effects
+			(font
+				(size 1.778 1.5113)
+			)
+			(justify left bottom)
+		)
+	)
+	(text "Graphics"
+		(exclude_from_sim no)
+		(at 63.5 99.06 90)
+		(effects
+			(font
+				(size 1.778 1.5113)
+			)
+			(justify left bottom)
+		)
+	)
+	(text "Graphics"
+		(exclude_from_sim no)
+		(at 149.86 111.76 90)
+		(effects
+			(font
+				(size 1.778 1.5113)
+			)
+			(justify left bottom)
+		)
+	)
+	(text "When key state goes up,\ntoggle output"
+		(exclude_from_sim no)
+		(at 180.34 50.8 0)
+		(effects
+			(font
+				(size 1.778 1.5113)
+			)
+			(justify left bottom)
+		)
+	)
+	(text "Inspired by SX64 keyboard and discussions\nwith Steve Gray and Mike Naberezny"
+		(exclude_from_sim no)
+		(at 213.36 35.56 0)
+		(effects
+			(font
+				(size 2.54 2.159)
+			)
+			(justify left bottom)
+		)
+	)
+	(text "Graphics"
+		(exclude_from_sim no)
+		(at 279.4 78.74 0)
+		(effects
+			(font
+				(size 1.778 1.5113)
+			)
+			(justify left bottom)
+		)
+	)
+	(text "R1.2A:\n- add KEYLOCK_LED output"
+		(exclude_from_sim no)
+		(at 233.172 172.72 0)
+		(effects
+			(font
+				(size 2.54 2.54)
+			)
+			(justify left)
+		)
+	)
+	(text "On Steve's MX replacement keyboards,\nAlternate Shift Lock is on\n- R9/C1 for Business and\n- R3/C5 for Graphics\nOriginal left shift is:\n- R3/C7 for Business and\n- R8/C0 for Graphics\n(Note: count starts at zero, not one)"
+		(exclude_from_sim no)
+		(at 27.94 68.58 0)
+		(effects
+			(font
+				(size 1.778 1.5113)
+			)
+			(justify left bottom)
+		)
+	)
+	(text "Graphics"
+		(exclude_from_sim no)
+		(at 114.3 111.76 90)
+		(effects
+			(font
+				(size 1.778 1.5113)
+			)
+			(justify left bottom)
+		)
+	)
+	(text "Business"
+		(exclude_from_sim no)
+		(at 279.4 127 0)
+		(effects
+			(font
+				(size 1.778 1.5113)
+			)
+			(justify left bottom)
+		)
+	)
 	(junction
 		(at 43.18 91.44)
@@
 		)
 	)
-	(text "Commodore PET SHIFT-LOCK simulator + RESET on long push"
-		(exclude_from_sim no)
-		(at 22.86 33.02 0)
-		(effects
-			(font
-				(size 3.81 3.2385)
-			)
-			(justify left bottom)
-		)
-	)
-	(text "CBM-ULTIPET-V1.2A"
-		(exclude_from_sim no)
-		(at 25.4 160.02 0)
-		(effects
-			(font
-				(size 3.81 3.2385)
-			)
-			(justify left bottom)
-		)
-	)
-	(text "Business"
-		(exclude_from_sim no)
-		(at 78.74 99.06 90)
-		(effects
-			(font
-				(size 1.778 1.5113)
-			)
-			(justify left bottom)
-		)
-	)
-	(text "Business"
-		(exclude_from_sim no)
-		(at 129.54 111.76 90)
-		(effects
-			(font
-				(size 1.778 1.5113)
-			)
-			(justify left bottom)
-		)
-	)
-	(text "Business"
-		(exclude_from_sim no)
-		(at 165.1 111.76 90)
-		(effects
-			(font
-				(size 1.778 1.5113)
-			)
-			(justify left bottom)
-		)
-	)
-	(text "Low = no key,\nhigh = key pressed"
-		(exclude_from_sim no)
-		(at 142.24 134.62 0)
-		(effects
-			(font
-				(size 1.778 1.5113)
-			)
-			(justify left bottom)
-		)
-	)
-	(text "Business"
-		(exclude_from_sim no)
-		(at 287.02 104.14 90)
-		(effects
-			(font
-				(size 1.778 1.5113)
-			)
-			(justify left bottom)
-		)
-	)
-	(text "Graphics"
-		(exclude_from_sim no)
-		(at 271.78 104.14 90)
-		(effects
-			(font
-				(size 1.778 1.5113)
-			)
-			(justify left bottom)
-		)
-	)
-	(text "/RES is 3.3V from CPU\nside. That then triggers\n/BRES on 5V side"
-		(exclude_from_sim no)
-		(at 195.58 137.16 0)
-		(effects
-			(font
-				(size 1.778 1.5113)
-			)
-			(justify left bottom)
-		)
-	)
-	(text "CBM-ULTIPET-1.2A-20241010"
-		(exclude_from_sim no)
-		(at 25.4 177.8 0)
-		(effects
-			(font
-				(size 2.54 2.159)
-			)
-			(justify left bottom)
-		)
-	)
-	(text "Saves the last\nkey press state"
-		(exclude_from_sim no)
-		(at 101.6 55.88 0)
-		(effects
-			(font
-				(size 1.778 1.5113)
-			)
-			(justify left bottom)
-		)
-	)
-	(text "Graphics"
-		(exclude_from_sim no)
-		(at 63.5 99.06 90)
-		(effects
-			(font
-				(size 1.778 1.5113)
-			)
-			(justify left bottom)
-		)
-	)
-	(text "Graphics"
-		(exclude_from_sim no)
-		(at 149.86 111.76 90)
-		(effects
-			(font
-				(size 1.778 1.5113)
-			)
-			(justify left bottom)
-		)
-	)
-	(text "When key state goes up,\ntoggle output"
-		(exclude_from_sim no)
-		(at 180.34 50.8 0)
-		(effects
-			(font
-				(size 1.778 1.5113)
-			)
-			(justify left bottom)
-		)
-	)
-	(text "Inspired by SX64 keyboard and discussions\nwith Steve Gray and Mike Naberezny"
-		(exclude_from_sim no)
-		(at 213.36 35.56 0)
-		(effects
-			(font
-				(size 2.54 2.159)
-			)
-			(justify left bottom)
-		)
-	)
-	(text "Graphics"
-		(exclude_from_sim no)
-		(at 279.4 78.74 0)
-		(effects
-			(font
-				(size 1.778 1.5113)
-			)
-			(justify left bottom)
-		)
-	)
-	(text "R1.2A:\n- add KEYLOCK_LED output"
-		(exclude_from_sim no)
-		(at 233.172 172.72 0)
-		(effects
-			(font
-				(size 2.54 2.54)
-			)
-			(justify left)
-		)
-	)
-	(text "On Steve's MX replacement keyboards,\nAlternate Shift Lock is on\n- R9/C1 for Business and\n- R3/C5 for Graphics\nOriginal left shift is:\n- R3/C7 for Business and\n- R8/C0 for Graphics\n(Note: count starts at zero, not one)"
-		(exclude_from_sim no)
-		(at 27.94 68.58 0)
-		(effects
-			(font
-				(size 1.778 1.5113)
-			)
-			(justify left bottom)
-		)
-	)
-	(text "Graphics"
-		(exclude_from_sim no)
-		(at 114.3 111.76 90)
-		(effects
-			(font
-				(size 1.778 1.5113)
-			)
-			(justify left bottom)
-		)
-	)
-	(text "Business"
-		(exclude_from_sim no)
-		(at 279.4 127 0)
-		(effects
-			(font
-				(size 1.778 1.5113)
-			)
-			(justify left bottom)
-		)
-	)
 	(label "ROW3"
 		(at 144.78 119.38 0)
@@
 			)
 		)
-		(property "Footprint" "cbm_ultipet_v1:DIL14"
+		(property "Footprint" "Package_DIP:DIP-14_W7.62mm_Socket_LongPads"
 			(at 111.76 68.58 0)
 			(effects
@@
 			)
 		)
-		(property "Footprint" "cbm_ultipet_v1:DIL14"
+		(property "Footprint" "Package_DIP:DIP-14_W7.62mm_Socket_LongPads"
 			(at 52.07 82.55 0)
 			(effects
@@
 			)
 		)
-		(property "Footprint" "cbm_ultipet_v1:DIL14"
+		(property "Footprint" "Package_DIP:DIP-14_W7.62mm_Socket_LongPads"
 			(at 157.48 157.48 0)
 			(effects
@@
 			)
 		)
-		(property "Footprint" "cbm_ultipet_v1:DIL14"
+		(property "Footprint" "Package_DIP:DIP-14_W7.62mm_Socket_LongPads"
 			(at 144.78 71.12 0)
 			(effects
@@
 			)
 		)
-		(property "Footprint" "cbm_ultipet_v1:DIL16"
+		(property "Footprint" "Package_DIP:DIP-16_W7.62mm_Socket_LongPads"
 			(at 43.18 83.82 0)
 			(effects
@@
 			)
 		)
-		(property "Footprint" "cbm_ultipet_v1:DIL14"
+		(property "Footprint" "Package_DIP:DIP-14_W7.62mm_Socket_LongPads"
 			(at 187.96 68.58 0)
 			(effects
@@
 			)
 		)
-		(property "Footprint" "cbm_ultipet_v1:DIL16"
+		(property "Footprint" "Package_DIP:DIP-16_W7.62mm_Socket_LongPads"
 			(at 86.36 124.46 0)
 			(effects

Commit message: more work on r1.3
Changed lines of the file:
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@@
+	(wire
+		(pts
+			(xy 82.55 41.91) (xy 86.36 41.91)
+		)
+		(stroke
+			(width 0.1524)
+			(type solid)
+		)
+	)
 	(wire
 		(pts
@@
 	(wire
 		(pts
-			(xy 86.36 63.5) (xy 86.36 45.72)
-		)
-		(stroke
-			(width 0.1524)
-			(type solid)
-		)
-	)
-	(wire
-		(pts
 			(xy 177.8 167.64) (xy 177.8 162.56)
 		)
@@
 		)
 	)
+	(wire
+		(pts
+			(xy 86.36 41.91) (xy 86.36 63.5)
+		)
+		(stroke
+			(width 0.1524)
+			(type solid)
+		)
+	)
 	(bus
 		(pts
@@
 	(wire
 		(pts
-			(xy 281.94 121.92) (xy 287.02 121.92)
+			(xy 281.94 121.92) (xy 284.48 121.92)
 		)
 		(stroke
@@
 	(wire
 		(pts
-			(xy 269.24 83.82) (xy 287.02 83.82)
+			(xy 269.24 83.82) (xy 281.94 83.82)
 		)
 		(stroke
@@
 	(wire
 		(pts
-			(xy 205.74 142.24) (xy 193.04 142.24)
-		)
-		(stroke
-			(width 0.1524)
-			(type solid)
-		)
-	)
-	(wire
-		(pts
 			(xy 167.64 71.12) (xy 175.26 71.12)
-		)
-		(stroke
-			(width 0.1524)
-			(type solid)
-		)
-	)
-	(wire
-		(pts
-			(xy 86.36 45.72) (xy 73.66 45.72)
 		)
 		(stroke
@@
 	(wire
 		(pts
+			(xy 209.55 142.24) (xy 205.74 142.24)
+		)
+		(stroke
+			(width 0.1524)
+			(type solid)
+		)
+	)
+	(wire
+		(pts
 			(xy 99.06 121.92) (xy 154.94 121.92)
 		)
@@
 	(global_label "/RES"
 		(shape bidirectional)
-		(at 200.66 142.24 0)
+		(at 209.55 142.24 0)
 		(fields_autoplaced yes)
 		(effects
@@
 		)
 		(property "Intersheetrefs" "${INTERSHEET_REFS}"
-			(at 209.5341 142.24 0)
+			(at 218.4241 142.24 0)
 			(effects
 				(font
@@
 	(global_label "/BRES"
 		(shape bidirectional)
-		(at 76.2 45.72 0)
+		(at 82.55 41.91 180)
 		(fields_autoplaced yes)
 		(effects
@@
 				(size 1.2446 1.2446)
 			)
-			(justify left)
+			(justify right)
 		)
 		(property "Intersheetrefs" "${INTERSHEET_REFS}"
-			(at 86.3187 45.72 0)
+			(at 72.4313 41.91 0)
 			(effects
 				(font
 					(size 1.27 1.27)
 				)
-				(justify left)
+				(justify right)
 				(hide yes)
 			)
@@
 	(global_label "KI0"
 		(shape bidirectional)
-		(at 274.32 83.82 0)
+		(at 281.94 83.82 0)
 		(fields_autoplaced yes)
 		(effects
@@
 		)
 		(property "Intersheetrefs" "${INTERSHEET_REFS}"
-			(at 281.3568 83.82 0)
+			(at 288.9768 83.82 0)
 			(effects
 				(font
@@
 	(global_label "/BRES"
 		(shape bidirectional)
-		(at 180.34 88.9 0)
+		(at 190.5 88.9 0)
 		(fields_autoplaced yes)
 		(effects
@@
 		)
 		(property "Intersheetrefs" "${INTERSHEET_REFS}"
-			(at 190.4587 88.9 0)
+			(at 200.6187 88.9 0)
 			(effects
 				(font

Commit message: preview for r1.3
Other:
- note added: "CBM-ULTIPET-V1.3A"
- note removed: "CBM-ULTIPET-V1.2A"
Changed lines of the file:
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@@
 		)
 	)
-	(text "CBM-ULTIPET-V1.2A"
+	(text "CBM-ULTIPET-V1.3A"
 		(exclude_from_sim no)
 		(at 25.4 160.02 0)

Commit message: some layout fixes, more parts
Parts:
- C130: footprint cbm_ultipet_v1:E2-4 -> cbm_ultipet_v1:E2-5
Changed lines of the file:
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@@
 			)
 		)
-		(property "Footprint" "cbm_ultipet_v1:E2-4"
+		(property "Footprint" "cbm_ultipet_v1:E2-5"
 			(at 177.8 170.18 0)
 			(effects
