File: Board/SID_Power.kicad_sch (KiCad schematic)
At the start: 12 parts

Commit message: ultipet 1.1a board
Parts:
- L4: value 170-200uH -> 200uH
Other:
- note added: "CBM-ULTIPET-V1.1A"
- note removed: "CBM-ULTIPET-V1.0A"
Changed lines of the file:
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@@
 		)
 	)
-	(text "CBM-ULTIPET-V1.0A"
+	(text "CBM-ULTIPET-V1.1A"
 		(exclude_from_sim no)
 		(at 170.18 142.24 0)
@@
 			)
 		)
-		(property "Value" "170-200uH"
+		(property "Value" "200uH"
 			(at 88.9 54.61 90)
 			(effects

Commit message: work on 1.3
Changed lines of the file:
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@@
 (kicad_sch
-	(version 20231120)
+	(version 20250114)
 	(generator "eeschema")
-	(generator_version "8.0")
+	(generator_version "9.0")
 	(paper "A4")
+	(text "CSA-DUALSID-1.0B-20231212"
+		(exclude_from_sim no)
+		(at 167.64 165.1 0)
+		(effects
+			(font
+				(size 2.54 2.159)
+			)
+			(justify left bottom)
+		)
+	)
+	(text "Vout = 12V -> RS/RG = 8.6\n-> RG=1.2k, RS=10k"
+		(exclude_from_sim no)
+		(at 111.76 157.48 0)
+		(effects
+			(font
+				(size 1.778 1.5113)
+			)
+			(justify left bottom)
+		)
+	)
+	(text "Vout = 9V -> RS/RG = 6.2\n-> RG=1.1k, RS=6.8k"
+		(exclude_from_sim no)
+		(at 111.76 149.86 0)
+		(effects
+			(font
+				(size 1.778 1.5113)
+			)
+			(justify left bottom)
+		)
+	)
+	(text "(C) A. Fachat"
+		(exclude_from_sim no)
+		(at 170.18 147.32 0)
+		(effects
+			(font
+				(size 2.54 2.159)
+			)
+			(justify left bottom)
+		)
+	)
+	(text "CBM-ULTIPET-V1.1A"
+		(exclude_from_sim no)
+		(at 170.18 142.24 0)
+		(effects
+			(font
+				(size 3.81 3.2385)
+			)
+			(justify left bottom)
+		)
+	)
+	(text "9V is not only used by SID\nbut also by Tape"
+		(exclude_from_sim no)
+		(at 111.76 167.64 0)
+		(effects
+			(font
+				(size 1.778 1.5113)
+			)
+			(justify left bottom)
+		)
+	)
+	(text "Vout=1.25 x (1 + RS/RG)"
+		(exclude_from_sim no)
+		(at 71.12 147.32 0)
+		(effects
+			(font
+				(size 1.778 1.5113)
+			)
+			(justify left bottom)
+		)
+	)
+	(text "V1.0B:\n- Fix parts footprint for L4, D2 and some caps"
+		(exclude_from_sim no)
+		(at 195.58 129.54 0)
+		(effects
+			(font
+				(size 1.9304 1.6408)
+			)
+			(justify left bottom)
+		)
+	)
+	(text "RS/RG = (Vout / 1.25) - 1"
+		(exclude_from_sim no)
+		(at 71.12 152.4 0)
+		(effects
+			(font
+				(size 1.778 1.5113)
+			)
+			(justify left bottom)
+		)
+	)
 	(junction
 		(at 111.76 76.2)
@@
 		)
 	)
-	(text "CSA-DUALSID-1.0B-20231212"
-		(exclude_from_sim no)
-		(at 167.64 165.1 0)
-		(effects
-			(font
-				(size 2.54 2.159)
-			)
-			(justify left bottom)
-		)
-	)
-	(text "Vout = 12V -> RS/RG = 8.6\n-> RG=1.2k, RS=10k"
-		(exclude_from_sim no)
-		(at 111.76 157.48 0)
-		(effects
-			(font
-				(size 1.778 1.5113)
-			)
-			(justify left bottom)
-		)
-	)
-	(text "Vout = 9V -> RS/RG = 6.2\n-> RG=1.1k, RS=6.8k"
-		(exclude_from_sim no)
-		(at 111.76 149.86 0)
-		(effects
-			(font
-				(size 1.778 1.5113)
-			)
-			(justify left bottom)
-		)
-	)
-	(text "(C) A. Fachat"
-		(exclude_from_sim no)
-		(at 170.18 147.32 0)
-		(effects
-			(font
-				(size 2.54 2.159)
-			)
-			(justify left bottom)
-		)
-	)
-	(text "CBM-ULTIPET-V1.1A"
-		(exclude_from_sim no)
-		(at 170.18 142.24 0)
-		(effects
-			(font
-				(size 3.81 3.2385)
-			)
-			(justify left bottom)
-		)
-	)
-	(text "9V is not only used by SID\nbut also by Tape"
-		(exclude_from_sim no)
-		(at 111.76 167.64 0)
-		(effects
-			(font
-				(size 1.778 1.5113)
-			)
-			(justify left bottom)
-		)
-	)
-	(text "Vout=1.25 x (1 + RS/RG)"
-		(exclude_from_sim no)
-		(at 71.12 147.32 0)
-		(effects
-			(font
-				(size 1.778 1.5113)
-			)
-			(justify left bottom)
-		)
-	)
-	(text "V1.0B:\n- Fix parts footprint for L4, D2 and some caps"
-		(exclude_from_sim no)
-		(at 195.58 129.54 0)
-		(effects
-			(font
-				(size 1.9304 1.6408)
-			)
-			(justify left bottom)
-		)
-	)
-	(text "RS/RG = (Vout / 1.25) - 1"
-		(exclude_from_sim no)
-		(at 71.12 152.4 0)
-		(effects
-			(font
-				(size 1.778 1.5113)
-			)
-			(justify left bottom)
-		)
-	)

Commit message: work on r1.3
Parts:
- U$24: footprint cbm_ultipet_v1:DIL08 -> Package_DIP:DIP-8_W7.62mm_Socket_LongPads
Changed lines of the file:
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@@
 			)
 		)
-		(property "Footprint" "cbm_ultipet_v1:DIL08"
+		(property "Footprint" "Package_DIP:DIP-8_W7.62mm_Socket_LongPads"
 			(at 73.66 83.82 0)
 			(effects

Commit message: preview for r1.3
Other:
- note added: "CBM-ULTIPET-V1.3A"
- note removed: "CBM-ULTIPET-V1.1A"
Changed lines of the file:
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@@
 		)
 	)
-	(text "CBM-ULTIPET-V1.1A"
+	(text "CBM-ULTIPET-V1.3A"
 		(exclude_from_sim no)
 		(at 170.18 142.24 0)

Commit message: more layout work on r1.3
Parts:
- added C168: 4700u, Capacitor_THT:CP_Radial_D16.0mm_P7.50mm, symbol Device:C_Polarized
- C97: value 100u -> 470u
Connections:
- net GND: now also C168.2
- net VCC: now also C168.1
Other:
- note added: "CSA-DUALSID-1.3A-20250807"
- note added: "V1.0B: - Fix parts footprint for L4, D2 and some caps V1.3A: - add large bypass cap at VCC entry - separate 9V VCC/GND from rest in layout to avoid audio interference"
- note removed: "CSA-DUALSID-1.0B-20231212"
- note removed: "V1.0B: - Fix parts footprint for L4, D2 and some caps"
- moved on the sheet: C98, C99, L2, RG0, RS0

Commit message: rename U refs to UX*
Parts:
- renumbered U$24 to UX24
Changed lines of the file:
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@@
 		(on_board yes)
 		(dnp no)
-		(property "Reference" "U$24"
+		(property "Reference" "UX24"
 			(at 78.74 66.04 0)
 			(effects
@@
 			(project "cbm_ultipet_v1"
 				(path "/4dd2dd78-173f-4b46-8cce-4ed940435c94/b1d6461c-fcfa-4cb9-bb95-7518479f88d1"
-					(reference "U$24")
+					(reference "UX24")
 					(unit 1)
 				)

Commit message: some layout fixes, more parts
Parts:
- C98: footprint cbm_ultipet_v1:E2,5-7 -> cbm_ultipet_v1:E2-5
Changed lines of the file:
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@@
 			)
 		)
-		(property "Footprint" "cbm_ultipet_v1:E2,5-7"
+		(property "Footprint" "cbm_ultipet_v1:E2-5"
 			(at 190.5 88.9 0)
 			(effects
