File: Board/Smallbus.kicad_sch (KiCad schematic)
At the start: 3 parts

Commit message: some layout fixes, more parts
Parts:
- C140, C75: footprint cbm_ultipet_v1:E2,5-7 -> cbm_ultipet_v1:E2,5-6
Changed lines of the file:
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@@
 			)
 		)
-		(property "Footprint" "cbm_ultipet_v1:E2,5-7"
+		(property "Footprint" "cbm_ultipet_v1:E2,5-6"
 			(at 133.35 76.2 0)
 			(effects
@@
 			)
 		)
-		(property "Footprint" "cbm_ultipet_v1:E2,5-7"
+		(property "Footprint" "cbm_ultipet_v1:E2,5-6"
 			(at 161.29 73.66 0)
 			(effects
