File: Board/VRAM,_DAC.kicad_sch (KiCad schematic)
At the start: 5 parts, among them IC10 RAMSOCK32TO512KSOP

Commit message: ultipet 1.1a board
Other:
- note added: "CBM-ULTIPET-V1.1A"
- note removed: "CBM-ULTIPET-V1.0A"
Changed lines of the file:
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@@
 		)
 	)
-	(text "CBM-ULTIPET-V1.0A"
+	(text "CBM-ULTIPET-V1.1A"
 		(exclude_from_sim no)
 		(at 261.62 190.5 0)

Commit message: various fixes as documented in github issues
Parts:
- removed JP5: JP2E, cbm_ultipet_v1:JP2, symbol cbm_ultipet_v1-eagle-import:JP2E
Other:
- note added: "1.2A: - removed DAC output connector pins (already on SID page)"
- note added: "CBM-ULTIPET-V1.2A"
- note added: "CBM-ULTIPET-V1.2A-20241010"
- note removed: "CBM-ULTIPET-V1.0A-20240104"
- note removed: "CBM-ULTIPET-V1.1A"

Commit message: preview for r1.3
Other:
- note added: "CBM-ULTIPET-V1.3A"
- note removed: "CBM-ULTIPET-V1.2A"
Changed lines of the file:
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@@
 		)
 	)
-	(text "CBM-ULTIPET-V1.2A"
+	(text "CBM-ULTIPET-V1.3A"
 		(exclude_from_sim no)
 		(at 261.62 190.5 0)

Commit message: layout work on r1.3a
Parts:
- removed IC10: RAMSOCK32TO512KSOP, cbm_ultipet_v1:SOP32, symbol cbm_ultipet_v1-eagle-import:RAMSOCK32TO512KSOP
- added C165: 0.1u, Capacitor_SMD:C_0603_1608Metric, symbol Device:C_Small
- added IC10: 512k x8 10ns SRAM, Package_SO:TSOP-II-44_10.16x18.41mm_P0.8mm, symbol Memory_RAM:IS61C5128AL-10TLI
Connections:
- net GND: now also C165.2, IC10.12 (GND), IC10.34 (GND)
- net RAMA0: now also IC10.3 (A0)
- net RAMA1: now also IC10.4 (A1)
- net RAMA10: now also IC10.26 (A10)
- net RAMA11: now also IC10.27 (A11)
- net RAMA12: now also IC10.28 (A12)
- net RAMA13: now also IC10.29 (A13)
- net RAMA14: now also IC10.30 (A14)
- net RAMA15: now also IC10.38 (A15)
- net RAMA16: now also IC10.39 (A16)
- net RAMA17: now also IC10.40 (A17)
- net RAMA18: now also IC10.41 (A18)
- net RAMA2: now also IC10.5 (A2)
- net RAMA3: now also IC10.6 (A3)
- net RAMA4: now also IC10.7 (A4)
- net RAMA5: now also IC10.16 (A5)
- net RAMA6: now also IC10.17 (A6)
- net RAMA7: now also IC10.18 (A7)
- net RAMA8: now also IC10.19 (A8)
- net RAMA9: now also IC10.20 (A9)
- net RAMD0: now also IC10.9 (I/O0)
- net RAMD1: now also IC10.10 (I/O1)
- net RAMD2: now also IC10.13 (I/O2)
- net RAMD3: now also IC10.14 (I/O3)
- net RAMD4: now also IC10.31 (I/O4)
- net RAMD5: now also IC10.32 (I/O5)
- net RAMD6: now also IC10.35 (I/O6)
- net RAMD7: now also IC10.36 (I/O7)
- net V33: now also C165.1, IC10.11 (VDD), IC10.33 (VDD)
- new net /RAMCS: IC10.37 (~{OE}), IC10.8 (~{CE})
- new net /RAMWE: IC10.15 (~{WE})
Other:
- note added: "1.2A: - removed DAC output connector pins (already on SID page) 1.3A: - replace 5V SRAM with 3.3V type"
- note added: "CBM-ULTIPET-V1.3A-20250806"
- note removed: "1.2A: - removed DAC output connector pins (already on SID page)"
- note removed: "CBM-ULTIPET-V1.2A-20241010"
