File: sdcardext/sdcardext.kicad_sch (KiCad schematic)
At the start: 2 parts, among them J1 Micro_SD_Card_Det2

Commit message: add part#, pullup for CD
Parts:
- added R1: 10k, Resistor_SMD:R_0603_1608Metric_Pad0.98x0.95mm_HandSolder, symbol Device:R
Connections:
- net VCC: now also R1.1
- net at P10.6 (CD): now also J1.10 (DET_A), J1.9 (DET_B), R1.2
Changed lines of the file:
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@@
 		(color 0 0 0 0)
 	)
+	(junction
+		(at 113.03 80.645)
+		(diameter 0)
+		(color 0 0 0 0)
+	)
+	(junction
+		(at 144.145 99.06)
+		(diameter 0)
+		(color 0 0 0 0)
+	)
 	(wire
 		(pts
@@
 	(wire
 		(pts
+			(xy 102.87 80.645) (xy 113.03 80.645)
+		)
+		(stroke
+			(width 0)
+			(type default)
+		)
+	)
+	(wire
+		(pts
+			(xy 144.145 99.695) (xy 147.955 99.695)
+		)
+		(stroke
+			(width 0)
+			(type default)
+		)
+	)
+	(wire
+		(pts
 			(xy 102.87 84.455) (xy 124.46 84.455)
 		)
@@
 	(wire
 		(pts
+			(xy 116.84 80.645) (xy 116.84 99.06)
+		)
+		(stroke
+			(width 0)
+			(type default)
+		)
+	)
+	(wire
+		(pts
 			(xy 120.65 94.615) (xy 120.65 81.915)
 		)
@@
 	(wire
 		(pts
+			(xy 147.955 97.155) (xy 144.145 97.155)
+		)
+		(stroke
+			(width 0)
+			(type default)
+		)
+	)
+	(wire
+		(pts
 			(xy 80.645 86.995) (xy 73.025 86.995)
 		)
@@
 	(wire
 		(pts
+			(xy 113.03 80.645) (xy 116.84 80.645)
+		)
+		(stroke
+			(width 0)
+			(type default)
+		)
+	)
+	(wire
+		(pts
 			(xy 73.025 86.995) (xy 73.025 83.185)
 		)
@@
 	(wire
 		(pts
+			(xy 113.03 66.675) (xy 113.03 69.215)
+		)
+		(stroke
+			(width 0)
+			(type default)
+		)
+	)
+	(wire
+		(pts
 			(xy 78.105 79.375) (xy 78.105 81.915)
 		)
@@
 	(wire
 		(pts
+			(xy 144.145 99.06) (xy 144.145 99.695)
+		)
+		(stroke
+			(width 0)
+			(type default)
+		)
+	)
+	(wire
+		(pts
 			(xy 147.955 84.455) (xy 140.97 84.455)
 		)
@@
 	(wire
 		(pts
+			(xy 144.145 97.155) (xy 144.145 99.06)
+		)
+		(stroke
+			(width 0)
+			(type default)
+		)
+	)
+	(wire
+		(pts
 			(xy 123.19 94.615) (xy 147.955 94.615)
 		)
@@
 	(wire
 		(pts
+			(xy 116.84 99.06) (xy 144.145 99.06)
+		)
+		(stroke
+			(width 0)
+			(type default)
+		)
+	)
+	(wire
+		(pts
 			(xy 120.65 81.915) (xy 147.955 81.915)
 		)
@@
 		(pts
 			(xy 125.73 97.155) (xy 102.87 97.155)
+		)
+		(stroke
+			(width 0)
+			(type default)
+		)
+	)
+	(wire
+		(pts
+			(xy 113.03 76.835) (xy 113.03 80.645)
 		)
 		(stroke
@@
 	)
 	(symbol
+		(lib_id "Device:R")
+		(at 113.03 73.025 0)
+		(unit 1)
+		(exclude_from_sim no)
+		(in_bom yes)
+		(on_board yes)
+		(dnp no)
+		(fields_autoplaced yes)
+		(property "Reference" "R1"
+			(at 115.57 71.7549 0)
+			(effects
+				(font
+					(size 1.27 1.27)
+				)
+				(justify left)
+			)
+		)
+		(property "Value" "10k"
+			(at 115.57 74.2949 0)
+			(effects
+				(font
+					(size 1.27 1.27)
+				)
+				(justify left)
+			)
+		)
+		(property "Footprint" "Resistor_SMD:R_0603_1608Metric_Pad0.98x0.95mm_HandSolder"
+			(at 111.252 73.025 90)
+			(effects
+				(font
+					(size 1.27 1.27)
+				)
+				(hide yes)
+			)
+		)
+		(property "Datasheet" "~"
+			(at 113.03 73.025 0)
+			(effects
+				(font
+					(size 1.27 1.27)
+				)
+				(hide yes)
+			)
+		)
+		(property "Description" "Resistor"
+			(at 113.03 73.025 0)
+			(effects
+				(font
+					(size 1.27 1.27)
+				)
+				(hide yes)
+			)
+		)
+		(pin "2"
+		)
+		(pin "1"
+		)
+		(instances
+			(project ""
+				(path "/a7752cdf-2a3d-405a-a832-a91866281276"
+					(reference "R1")
+					(unit 1)
+				)
+			)
+		)
+	)
+	(symbol
 		(lib_id "power:GNDD")
 		(at 140.97 102.87 0)
@@
 					(unit 1)
 				)
+			)
+		)
+	)
+	(symbol
+		(lib_id "power:VCC")
+		(at 113.03 66.675 0)
+		(unit 1)
+		(exclude_from_sim no)
+		(in_bom yes)
+		(on_board yes)
+		(dnp no)
+		(fields_autoplaced yes)
+		(property "Reference" "#PWR05"
+			(at 113.03 70.485 0)
+			(effects
+				(font
+					(size 1.27 1.27)
+				)
+				(hide yes)
+			)
+		)
+		(property "Value" "VCC"
+			(at 113.03 61.595 0)
+			(effects
+				(font
+					(size 1.27 1.27)
+				)
+			)
+		)
+		(property "Footprint" ""
+			(at 113.03 66.675 0)
+			(effects
+				(font
+					(size 1.27 1.27)
+				)
+				(hide yes)
+			)
+		)
+		(property "Datasheet" ""
+			(at 113.03 66.675 0)
+			(effects
+				(font
+					(size 1.27 1.27)
+				)
+				(hide yes)
+			)
+		)
+		(property "Description" "Power symbol creates a global label with name \"VCC\""
+			(at 113.03 66.675 0)
+			(effects
+				(font
+					(size 1.27 1.27)
+				)
+				(hide yes)
+			)
+		)
+		(pin "1"
+		)
+		(instances
+			(project "sdcardext"
+				(path "/a7752cdf-2a3d-405a-a832-a91866281276"
+					(reference "#PWR05")
+					(unit 1)
+				)

Commit message: SD card and volumn poti test extension
Parts:
- added C1: 100u, Capacitor_SMD:C_1206_3216Metric_Pad1.33x1.80mm_HandSolder, symbol Device:C_Polarized
- added C2: 100n, Capacitor_SMD:C_0603_1608Metric_Pad1.08x0.95mm_HandSolder, symbol Device:C
- added J2: Conn_02x03_Odd_Even, Connector_IDC:IDC-Header_2x03_P2.54mm_Horizontal, symbol Connector_Generic:Conn_02x03_Odd_Even
- added RV1: R_Potentiometer_Dual, Potentiometer_THT:Potentiometer_Alps_RK097_Dual_Horizontal_Switch, symbol Device:R_Potentiometer_Dual
- J1: LCSC (none) -> C585350
- P10: footprint Connector_IDC:IDC-Header_2x06_P2.54mm_Vertical -> Connector_IDC:IDC-Header_2x06_P2.54mm_Horizontal; LCSC (none) -> C9141
- R1: LCSC (none) -> C25804
Connections:
- net GNDD: now also C1.2, C2.2
- net VCC: now also C1.1, C2.1
- new net: J2.5 (Pin_5), RV1.1
- new net: J2.3 (Pin_3), RV1.2
- new net: J2.1 (Pin_1), RV1.3
- new net: J2.2 (Pin_2), RV1.4
- new net: J2.4 (Pin_4), RV1.5
- new net: J2.6 (Pin_6), RV1.6
Other:
- moved on the sheet: J1, P10, R1
