File: HDMItest2/HDMItest.kicad_pcb (KiCad board)
At the start: 2 copper layers, 54.1 x 29 mm, 43 parts, among them J1 HDMI_A, J2 Conn_02x06_Odd_Even

Commit message: move sdcard to pcb_bits
Parts:
- U1: footprint Package_DFN_QFN:Texas_RNQ0040A_WQFN-40-1EP_6x4mm_P0.4mm_EP4.7x2.7mm_ThermalVias -> Package_DFN_QFN:QFN-40-1EP_5x5mm_P0.4mm_EP3.8x3.8mm_ThermalVias
Routing:
- net GND: track 75.8 -> 80.9 mm, vias 11 -> 12
- net Net-(JP10-B): track 144.6 -> 147.2 mm
- net Net-(J1-D2+): track 6.95 -> 5.98 mm
- net Net-(U1-IN_C_B): track 6.07 -> 5.13 mm
- net Net-(J1-SCL): track 29.4 -> 28.6 mm
- net Net-(JP3-B): track 24.3 -> 23.6 mm
- net Net-(JP4-B): track 6.32 -> 5.62 mm
- net Net-(J1-SDA): track 35.5 -> 34.8 mm
- net Net-(JP2-B): track 11.6 -> 10.9 mm
- net Net-(J1-D1-): track 4.97 -> 5.61 mm
- net Net-(U1-IN_D3_B): track 3.66 -> 4.30 mm
- net Net-(J1-CK-): track 4.55 -> 5.19 mm
- net Net-(J1-D0+): track 4.93 -> 5.57 mm
- net Net-(J1-CK+): track 4.80 -> 5.44 mm
- net Net-(J1-D0-): track 4.68 -> 5.32 mm
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