File: HDMItest2/HDMItest.kicad_sch (KiCad schematic)
At the start: 43 parts, among them J1 HDMI_A, J2 Conn_02x06_Odd_Even

Commit message: move sdcard to pcb_bits
Parts:
- P11: value ~ -> (none)
- U1: value ~ -> (none); footprint Package_DFN_QFN:Texas_RNQ0040A_WQFN-40-1EP_6x4mm_P0.4mm_EP4.7x2.7mm_ThermalVias -> Package_DFN_QFN:QFN-40-1EP_5x5mm_P0.4mm_EP3.8x3.8mm_ThermalVias
